File: PowerPack.kicad_sch (KiCad schematic)
At the start: 75 parts, among them CN1 XT30PW-M, Q1 NTMFS5C670NLT1G, Q2 NTMFS5C670NLT1G, Q3 NTMFS5C670NLT1G, Q4 NTMFS5C670NLT1G, Q5 2N7002, Q6 2301_C334113, Q7 2301_C334113, Q8 2N7002, Q9 WSD3066DN33, U1 IP2368_BZ_VGLIP_C5203723, U2 22uF, U3 22uF, U4 22uF, U5 22uF, U6 22uF, U7 22uF, U8 ME6203A50PG

Commit message: start pcb design
Parts:
- removed C1: 220uF, easyeda2kicad:CAP-TH_BD8.0-P3.50-D0.6-FD, symbol easyeda2kicad:SPZ1VM221F11O00RAXXX
- added CR1: 220uF, easyeda2kicad:CAP-TH_BD8.0-P3.50-D0.6-FD, symbol easyeda2kicad:SPZ1VM221F11O00RAXXX
- C3: renamed from C5; footprint (none) -> Capacitor_SMD:C_0402_1005Metric_Pad0.74x0.62mm_HandSolder
- C4: renamed from C6; footprint (none) -> Capacitor_SMD:C_0402_1005Metric_Pad0.74x0.62mm_HandSolder
- renumbered C19 to C10, C18 to C11, C20 to C12, C21 to C13, C7 to C2, C8 to C5, C14 to C6, C15 to C7, C16 to C8, C17 to C9, C2 to CL1, U4 to CL2, U3 to CL3, U2 to CL4, C4 to CL7, C10 to CLQ1, C9 to CLQ2, U7 to CR2, U6 to CR3, U5 to CR4, C12 to CRQ1, C13 to CRQ2, C11 to CSC1, JP3 to JP1, JP1 to JP2, Q9 to Q1, Q6 to QE1, Q7 to QE2, Q8 to QE3, Q5 to QE4, Q3 to QLB1, Q1 to QLT1, Q4 to QRB1, Q2 to QRT1, R9 to R1, R4 to R10, R20 to R12, R21 to R13, R19 to R14, R18 to R15, R17 to R16, R12 to R17, R13 to R18, R16 to R19, R10 to R2, R15 to R20, R14 to R21, R25 to R22, R24 to R23, R27 to R24, R26 to R25, R23 to R4, R7 to R5, R5 to R6, R22 to R7, R6 to R8, R8 to R9, RNTC to RNTC1, U8 to U2
Connections:
- net GND: now also CL1.2, CR1.2; no longer CL1.1
- net VBUSL_Source: now also CL1.1; no longer CL1.2
- net VBUSR_Source: now also CR1.1
Other:
- moved on the sheet: CL1

Commit message: route pcb
Parts:
- C12, C13: value 100nf -> 100nf
Connections:
- net BAT-MODE: now also R13.1, U1.46 (BAT_MODE); no longer JP2.1 (A), R13.2
- net ISET-MODE: no longer names the net of JP1.1 (A), R12.2
- new net: JP2.1 (A), R13.2
Other:
- moved on the sheet: R12, R13
Changed lines of the file:
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@@
 (kicad_sch
-	(version 20231120)
+	(version 20250114)
 	(generator "eeschema")
-	(generator_version "8.0")
+	(generator_version "9.0")
 	(paper "A3")
 	(title_block
 		(title "PowerPack")
 	)
+	(text "5S"
+		(exclude_from_sim no)
+		(at 249.174 177.292 0)
+		(effects
+			(font
+				(size 1.27 1.27)
+			)
+		)
+	)
+	(text "6S"
+		(exclude_from_sim no)
+		(at 248.92 184.912 0)
+		(effects
+			(font
+				(size 1.27 1.27)
+			)
+		)
+	)
+	(text "4S"
+		(exclude_from_sim no)
+		(at 249.174 169.672 0)
+		(effects
+			(font
+				(size 1.27 1.27)
+			)
+		)
+	)
 	(junction
 		(at 40.64 242.57)
@@
 	)
 	(junction
-		(at 226.06 138.43)
-		(diameter 0)
-		(color 0 0 0 0)
-	)
-	(junction
 		(at 332.74 46.99)
 		(diameter 0)
@@
 	)
 	(junction
-		(at 226.06 135.89)
-		(diameter 0)
-		(color 0 0 0 0)
-	)
-	(junction
 		(at 88.9 252.73)
 		(diameter 0)
@@
 	)
 	(junction
+		(at 218.44 138.43)
+		(diameter 0)
+		(color 0 0 0 0)
+	)
+	(junction
 		(at 88.9 229.87)
 		(diameter 0)
@@
 	(wire
 		(pts
+			(xy 227.33 135.89) (xy 238.76 135.89)
+		)
+		(stroke
+			(width 0)
+			(type default)
+		)
+	)
+	(wire
+		(pts
 			(xy 113.03 266.7) (xy 111.76 266.7)
 		)
@@
 	(wire
 		(pts
+			(xy 218.44 138.43) (xy 217.17 138.43)
+		)
+		(stroke
+			(width 0)
+			(type default)
+		)
+	)
+	(wire
+		(pts
 			(xy 393.7 25.4) (xy 393.7 35.56)
 		)
@@
 	(wire
 		(pts
-			(xy 226.06 138.43) (xy 224.79 138.43)
-		)
-		(stroke
-			(width 0)
-			(type default)
-		)
-	)
-	(wire
-		(pts
-			(xy 226.06 135.89) (xy 224.79 135.89)
-		)
-		(stroke
-			(width 0)
-			(type default)
-		)
-	)
-	(wire
-		(pts
 			(xy 166.37 231.14) (xy 166.37 254)
 		)
@@
 	(wire
 		(pts
-			(xy 238.76 135.89) (xy 226.06 135.89)
-		)
-		(stroke
-			(width 0)
-			(type default)
-		)
-	)
-	(wire
-		(pts
 			(xy 337.82 46.99) (xy 339.09 46.99)
 		)
@@
 	(wire
 		(pts
-			(xy 226.06 138.43) (xy 226.06 140.97)
-		)
-		(stroke
-			(width 0)
-			(type default)
-		)
-	)
-	(wire
-		(pts
 			(xy 40.64 161.29) (xy 40.64 163.83)
 		)
@@
 	(wire
 		(pts
+			(xy 218.44 142.24) (xy 218.44 138.43)
+		)
+		(stroke
+			(width 0)
+			(type default)
+		)
+	)
+	(wire
+		(pts
 			(xy 228.6 179.07) (xy 228.6 181.61)
 		)
@@
 	(wire
 		(pts
+			(xy 219.71 138.43) (xy 218.44 138.43)
+		)
+		(stroke
+			(width 0)
+			(type default)
+		)
+	)
+	(wire
+		(pts
 			(xy 52.07 242.57) (xy 63.5 242.57)
 		)
@@
 	(wire
 		(pts
+			(xy 227.33 142.24) (xy 218.44 142.24)
+		)
+		(stroke
+			(width 0)
+			(type default)
+		)
+	)
+	(wire
+		(pts
 			(xy 58.42 171.45) (xy 58.42 176.53)
 		)
@@
 	(wire
 		(pts
-			(xy 226.06 133.35) (xy 226.06 135.89)
-		)
-		(stroke
-			(width 0)
-			(type default)
-		)
-	)
-	(wire
-		(pts
 			(xy 248.92 171.45) (xy 251.46 171.45)
 		)
@@
 	(wire
 		(pts
+			(xy 219.71 135.89) (xy 217.17 135.89)
+		)
+		(stroke
+			(width 0)
+			(type default)
+		)
+	)
+	(wire
+		(pts
 			(xy 175.26 254) (xy 172.72 254)
 		)
@@
 	(wire
 		(pts
-			(xy 238.76 138.43) (xy 226.06 138.43)
+			(xy 227.33 138.43) (xy 238.76 138.43)
 		)
 		(stroke
@@
 		)
 	)
-	(text "5S"
-		(exclude_from_sim no)
-		(at 249.174 177.292 0)
-		(effects
-			(font
-				(size 1.27 1.27)
-			)
-		)
-	)
-	(text "6S"
-		(exclude_from_sim no)
-		(at 248.92 184.912 0)
-		(effects
-			(font
-				(size 1.27 1.27)
-			)
-		)
-	)
-	(text "4S"
-		(exclude_from_sim no)
-		(at 249.174 169.672 0)
-		(effects
-			(font
-				(size 1.27 1.27)
-			)
-		)
-	)
 	(global_label "HLED"
 		(shape input)
@@
 	(global_label "BAT-MODE"
 		(shape input)
-		(at 226.06 140.97 0)
+		(at 227.33 142.24 0)
 		(fields_autoplaced yes)
 		(effects
@@
 		)
 		(property "Intersheetrefs" "${INTERSHEET_REFS}"
-			(at 239.1447 140.97 0)
+			(at 240.4147 142.24 0)
 			(effects
 				(font
@@
 		)
 	)
-	(global_label "ISET-MODE"
-		(shape input)
-		(at 226.06 133.35 0)
-		(fields_autoplaced yes)
-		(effects
-			(font
-				(size 1.27 1.27)
-			)
-			(justify left)
-		)
-		(property "Intersheetrefs" "${INTERSHEET_REFS}"
-			(at 239.7494 133.35 0)
-			(effects
-				(font
-					(size 1.27 1.27)
-				)
-				(justify left)
-				(hide yes)
-			)
-		)
-	)
 	(global_label "VBUSL_CIO"
 		(shape input)
@@
 	(symbol
 		(lib_id "Device:R")
-		(at 220.98 135.89 90)
+		(at 223.52 135.89 90)
 		(unit 1)
 		(exclude_from_sim no)
@@
 		(dnp no)
 		(property "Reference" "R12"
-			(at 223.012 133.858 90)
+			(at 225.552 133.858 90)
 			(effects
 				(font
@@
 		)
 		(property "Value" "1k"
-			(at 222.25 135.89 90)
+			(at 224.79 135.89 90)
 			(effects
 				(font
@@
 		)
 		(property "Footprint" "Resistor_SMD:R_0402_1005Metric_Pad0.72x0.64mm_HandSolder"
-			(at 220.98 137.668 90)
+			(at 223.52 137.668 90)
 			(effects
 				(font
@@
 		)
 		(property "Datasheet" "~"
-			(at 220.98 135.89 0)
+			(at 223.52 135.89 0)
 			(effects
 				(font
@@
 		)
 		(property "Description" "Resistor"
-			(at 220.98 135.89 0)
+			(at 223.52 135.89 0)
 			(effects
 				(font
@@
 	(symbol
 		(lib_id "Device:R")
-		(at 220.98 138.43 90)
+		(at 223.52 138.43 90)
 		(unit 1)
 		(exclude_from_sim no)
@@
 		(dnp no)
 		(property "Reference" "R13"
-			(at 223.012 140.462 90)
+			(at 225.552 140.462 90)
 			(effects
 				(font
@@
 		)
 		(property "Value" "1k"
-			(at 222.25 138.43 90)
+			(at 224.79 138.43 90)
 			(effects
 				(font
@@
 		)
 		(property "Footprint" "Resistor_SMD:R_0402_1005Metric_Pad0.72x0.64mm_HandSolder"
-			(at 220.98 140.208 90)
+			(at 223.52 140.208 90)
 			(effects
 				(font
@@
 		)
 		(property "Datasheet" "~"
-			(at 220.98 138.43 0)
+			(at 223.52 138.43 0)
 			(effects
 				(font
@@
 		)
 		(property "Description" "Resistor"
-			(at 220.98 138.43 0)
+			(at 223.52 138.43 0)
 			(effects
 				(font
@@
 			)
 		)
-		(property "Value" "100nf "
+		(property "Value" "100nf"
 			(at 335.28 55.372 0)
 			(effects
@@
 			)
 		)
-		(property "Value" "100nf "
+		(property "Value" "100nf"
 			(at 375.92 57.912 0)
 			(effects
@@
 		)
 	)
+	(embedded_fonts no)
 )
