File: balancingBoard/balancingBoard.kicad_pcb (KiCad board)
At the start: 2 copper layers, 52 parts, among them CN1 WJ15EDGRC-3.81-4P, CN2 WJ15EDGRC-3.81-4P, CN3 XT30PW-M, CN4 XT30PW-M, Q1 IRFH5302TRPBF, Q3 IRFH5302TRPBF, U1 BQ7791502PWR, U2 BQ7791502PWR

Commit message: add layout for balancingboard
Parts:
- removed CN4: XT30PW-M, easyeda2kicad:CONN-TH_XT30PW-M
- added R18: 10k, Resistor_SMD:R_0603_1608Metric_Pad0.98x0.95mm_HandSolder, F.Cu at (121.0, 83.5)
- added U3: XT30PW-F, easyeda2kicad:CONN-TH_XT30PW-F-1, F.Cu at (121.5, 105.2)
- CN3: moved to F.Cu
- moved C53 63.6 mm to (104.2, 80.9), turned to -90 degrees
- moved C6 56.2 mm to (104.2, 67.1), turned to -90 degrees
- moved CN3 55.7 mm to (93.5, 105.2), turned to -90 degrees
- moved R6 35.9 mm to (116.0, 82.0), turned to 180 degrees
- moved R14 34.8 mm to (116.5, 91.0), turned to -90 degrees
- moved D2 32.4 mm to (118.0, 91.0), turned to 90 degrees
- moved R7 32.1 mm to (116.0, 80.5)
- moved R8 28.8 mm to (116.0, 83.5), turned to 180 degrees
- moved R11 26.4 mm to (116.0, 71.8), turned to 180 degrees
- moved R12 25.9 mm to (116.0, 73.2)
- moved R16 24.7 mm to (116.0, 74.8)
- moved R47 24.4 mm to (116.0, 86.0), turned to 180 degrees
- moved R48 24.1 mm to (116.0, 87.5), turned to 180 degrees
- moved R30 20.6 mm to (105.4, 91.1), turned to 90 degrees
- moved R15 19.7 mm to (123.5, 69.2), turned to 90 degrees
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Connections:
- CN1 pad 1: +BATT -> Net-(CN1-Pad1)
- CN3 pad 1: GND -> -BATT
- CN3 pad 2: +BATT -> PACK+
- CN3 pad 3: GND -> unconnected-(CN3-Pad3)
- CN3 pad 4: GND -> unconnected-(CN3-Pad4)
- Q3 pad 1: -BATT -> PACK-
- Q3 pad 2: -BATT -> PACK-
- Q3 pad 3: -BATT -> PACK-
- R1 pad 1: +BATT -> Net-(CN1-Pad1)
- R13 pad 1: GND -> -BATT
- R14 pad 2: -BATT -> PACK-
- R2 pad 1: +BATT -> Net-(CN1-Pad1)
- R31 pad 2: -BATT -> PACK-
- R34 pad 2: -BATT -> PACK-
- U1 pad 10: GND -> -BATT
Routing:
- net Net-(U1-SRN): track 0.00 -> 25.4 mm
- net Net-(U2-CTRC): track 0.00 -> 25.1 mm, vias 0 -> 4
- net Net-(D2-C): track 0.00 -> 24.2 mm, vias 0 -> 2
- net Net-(U2-VDD): track 0.00 -> 22.8 mm
- net BCBO: track 0.00 -> 18.9 mm, vias 0 -> 2
- net -BATT: track 0.00 -> 18.0 mm
- net Net-(U2-VC2): track 0.00 -> 15.9 mm
- net Net-(U2-VC3): track 0.00 -> 15.9 mm
- net Net-(U2-LPWR): track 0.00 -> 14.8 mm, vias 0 -> 2
- net Net-(U2-DSG): track 0.00 -> 13.3 mm
- net Net-(U2-TS): track 0.00 -> 12.6 mm
- net Net-(U1-TS): track 0.00 -> 12.2 mm
- net Net-(U2-VC1): track 0.00 -> 12.0 mm
- net PACK-: track 0.00 -> 11.7 mm
- net Net-(U1-VCO): track 0.00 -> 11.7 mm
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- added copper zone on F.Cu, net -BATT
- added copper zone on B.Cu, net GND
- added copper zone on F.Cu, net GND
- added copper zone on B.Cu, net Net-(Q1-D-Pad5)
- added copper zone on F.Cu, net Net-(Q1-D-Pad5)
- added copper zone on F.Cu, net Net-(U1-SRN)
- added copper zone on B.Cu, net Net-(U2-CTRC)
- added copper zone on F.Cu, net Net-(U2-CTRC)
- added copper zone on B.Cu, net PACK+
- added copper zone on F.Cu, net PACK+
- added copper zone on F.Cu, net PACK-
Other:
- board outline added: 40 x 56.2 mm
