File: balancingBoard/balancingBoard.kicad_pcb (KiCad board)
At the start: 2 copper layers, 40 x 56.2 mm, 53 parts, among them CN1 WJ15EDGRC-3.81-4P, CN2 WJ15EDGRC-3.81-4P, CN3 XT30PW-M, Q1 IRFH5302TRPBF, Q3 IRFH5302TRPBF, U1 BQ7791502PWR, U2 BQ7791502PWR, U3 XT30PW-F

Commit message: generate all boms
Parts:
- R11: value 100k -> 10M
Changed lines of the file:
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@@
 			)
 		)
-		(property "Value" "100k"
+		(property "Value" "10M"
 			(at 0 1.43 0)
 			(layer "F.Fab")

Commit message: add some more
Connections:
- C5 pad 2: Net-(U2-VDD) -> Net-(U2-CCFG)
- C52 pad 2: Net-(U1-VDD) -> Net-(U1-CCFG)
- R1 pad 2: Net-(U2-VDD) -> Net-(U2-CCFG)
- R36 pad 2: Net-(U1-VDD) -> Net-(U1-CCFG)
- R9 pad 2: Net-(U2-VDD) -> Net-(U2-CCFG)
- U1 pad 1: Net-(U1-VDD) -> Net-(U1-CCFG)
- U1 pad 20: Net-(U1-AVDD) -> Net-(U1-CCFG)
- U2 pad 1: Net-(U2-VDD) -> Net-(U2-CCFG)
- U2 pad 20: Net-(U2-AVDD) -> Net-(U2-CCFG)
Routing:
- net Net-(U2-CCFG): track 0.00 -> 29.5 mm
- net Net-(U2-VDD): track 22.8 -> 0.00 mm
- net Net-(U1-CCFG): track 0.00 -> 14.0 mm
- net Net-(U1-VDD): track 7.32 -> 0.00 mm
- net Net-(U2-AVDD): track 8.42 -> 2.05 mm
- net Net-(U1-AVDD): track 8.54 -> 2.17 mm
Other:
- board text added: "Janek"
- board text added: "github.com/janekc"
