File: balancingBoard/balancingBoard.kicad_sch (KiCad schematic)
At the start: 54 parts, among them Q1 IRFH5302TRPBF, Q3 IRFH5302TRPBF, U1 BQ7791502PWR, U2 BQ7791502PWR

Commit message: update#
Parts:
- removed D1: D, symbol Device:D
- added CN1, CN2: WJ15EDGRC-3.81-4P, easyeda2kicad:CONN-TH_WJ15EDGRC-3.81-4P, symbol easyeda2kicad:WJ15EDGRC-3.81-4P
- added CN3, CN4: XT30PW-M, easyeda2kicad:CONN-TH_XT30PW-M, symbol easyeda2kicad:XT30PW-M
- added D2: 1SS355, easyeda2kicad:SOD-323_L1.8-W1.3-LS2.5-RD, symbol easyeda2kicad:1SS355_C2892574
- R12, R8: value R -> 10k; footprint (none) -> Resistor_SMD:R_0603_1608Metric_Pad0.98x0.95mm_HandSolder
- R16: value R -> 1M; footprint (none) -> Resistor_SMD:R_0603_1608Metric_Pad0.98x0.95mm_HandSolder
- R6, R7: value R -> 10M; footprint (none) -> Resistor_SMD:R_0603_1608Metric_Pad0.98x0.95mm_HandSolder
Connections:
- net +BATT: now also CN1.1, CN3.2 (+), CN4.2 (+)
- net -BATT: now also CN4.1 (-)
- net GND: now also CN2.4, CN3.1 (-), CN3.3, CN3.4, CN4.3, CN4.4; no longer C3.2, C4.1
- net at BT1.2, BT2.1, R28.1: now also CN2.3
- net at BT2.2, BT3.1, R27.1: now also CN2.2
- net at BT3.2, BT6.1, C5.1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: now also C3.2, C4.1, CN1.4, CN2.1
- net at BT4.1, BT5.2, R3.1: now also CN1.2
- net at BT5.1, BT6.2, R4.1: now also CN1.3
- net at R14.1: now also D2.2 (A)
- net at R16.1, U2.14 (LD): now also D2.1 (C)
Other:
- moved on the sheet: BT1, BT2, BT3, BT4, BT5, BT6, C1, C2, C3, C4, C49, C5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

Commit message: add layout for balancingboard
Parts:
- removed CN4: XT30PW-M, easyeda2kicad:CONN-TH_XT30PW-M, symbol easyeda2kicad:XT30PW-M
- added R18: 10k, Resistor_SMD:R_0603_1608Metric_Pad0.98x0.95mm_HandSolder, symbol Device:R
- added U3: XT30PW-F, easyeda2kicad:CONN-TH_XT30PW-F-1, symbol easyeda2kicad:XT30PW-F
Connections:
- net +BATT: now also U3.1; no longer BT4.2, CN1.1, R1.1, R2.1
- net -BATT: now also CN3.1 (-), R13.1, U1.10 (SRP); no longer Q3.1 (S), Q3.2 (S), Q3.3 (S), R14.2, R31.2, R34.2
- net GND: now also R18.2; no longer CN3.1 (-), CN3.3, CN3.4, R13.1, U1.10 (SRP)
- net at R19.1, R21.2, U1.18 (TS): now also R18.1
- new net: BT4.2, CN1.1, R1.1, R2.1
- new net PACK-: Q3.1 (S), Q3.2 (S), Q3.3 (S), R14.2, R31.2, R34.2, U3.2
Other:
- note added: "CEL1"
- note added: "CEL2"
- note added: "CEL3"
- note added: "CEL4"
- note added: "CEL5"
- note added: "CEL6"
- moved on the sheet: CN2, CN3

Commit message: generate all boms
Parts:
- R11: value 100k -> 10M
Changed lines of the file:
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@@
 			)
 		)
-		(property "Value" "100k"
+		(property "Value" "10M"
 			(at 168.91 49.53 90)
 			(effects

Commit message: add some more
Connections:
- net at C52.2, R36.2, U1.1 (VDD): now also U1.20 (CCFG)
- net at C53.2, U1.2 (AVDD): no longer U1.20 (CCFG)
- net at C5.2, R1.2, R9.2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: now also U2.20 (CCFG)
- net at C6.2, U2.2 (AVDD): no longer U2.20 (CCFG)
Changed lines of the file:
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@@
+	)
+	(junction
+		(at 171.45 36.83)
+		(diameter 0)
+		(color 0 0 0 0)
 	)
 	(junction
@@
 	)
 	(junction
+		(at 135.89 102.87)
+		(diameter 0)
+		(color 0 0 0 0)
+	)
+	(junction
 		(at 100.33 88.9)
 		(diameter 0)
@@
 	)
 	(junction
-		(at 134.62 105.41)
-		(diameter 0)
-		(color 0 0 0 0)
-	)
-	(junction
 		(at 190.5 83.82)
 		(diameter 0)
@@
 	(junction
 		(at 119.38 52.07)
-		(diameter 0)
-		(color 0 0 0 0)
-	)
-	(junction
-		(at 134.62 34.29)
 		(diameter 0)
 		(color 0 0 0 0)
@@
 	(wire
 		(pts
-			(xy 134.62 105.41) (xy 139.7 105.41)
+			(xy 128.27 105.41) (xy 139.7 105.41)
 		)
 		(stroke
@@
 		(pts
 			(xy 172.72 118.11) (xy 162.56 118.11)
-		)
-		(stroke
-			(width 0)
-			(type default)
-		)
-	)
-	(wire
-		(pts
-			(xy 134.62 91.44) (xy 134.62 105.41)
 		)
 		(stroke
@@
 	(wire
 		(pts
-			(xy 134.62 20.32) (xy 134.62 34.29)
-		)
-		(stroke
-			(width 0)
-			(type default)
-		)
-	)
-	(wire
-		(pts
 			(xy 162.56 31.75) (xy 163.83 31.75)
 		)
@@
 	(wire
 		(pts
-			(xy 130.81 102.87) (xy 139.7 102.87)
+			(xy 130.81 102.87) (xy 135.89 102.87)
 		)
 		(stroke
@@
 	(wire
 		(pts
-			(xy 173.99 91.44) (xy 134.62 91.44)
-		)
-		(stroke
-			(width 0)
-			(type default)
-		)
-	)
-	(wire
-		(pts
-			(xy 134.62 34.29) (xy 139.7 34.29)
+			(xy 171.45 92.71) (xy 135.89 92.71)
 		)
 		(stroke
@@
 		)
 	)
-	(wire
-		(pts
-			(xy 128.27 105.41) (xy 134.62 105.41)
-		)
-		(stroke
-			(width 0)
-			(type default)
-		)
-	)
 	(polyline
 		(pts
@@
 	(wire
 		(pts
-			(xy 173.99 41.91) (xy 173.99 20.32)
-		)
-		(stroke
-			(width 0)
-			(type default)
-		)
-	)
-	(wire
-		(pts
 			(xy 185.42 149.86) (xy 185.42 147.32)
 		)
@@
 	(wire
 		(pts
+			(xy 162.56 41.91) (xy 171.45 41.91)
+		)
+		(stroke
+			(width 0)
+			(type default)
+		)
+	)
+	(wire
+		(pts
 			(xy 43.18 157.48) (xy 121.92 157.48)
 		)
@@
 	(wire
 		(pts
-			(xy 173.99 20.32) (xy 134.62 20.32)
-		)
-		(stroke
-			(width 0)
-			(type default)
-		)
-	)
-	(wire
-		(pts
 			(xy 139.7 110.49) (xy 137.16 110.49)
 		)
@@
 	(wire
 		(pts
-			(xy 162.56 113.03) (xy 173.99 113.03)
+			(xy 171.45 113.03) (xy 162.56 113.03)
 		)
 		(stroke
@@
 		(pts
 			(xy 160.02 154.94) (xy 160.02 157.48)
+		)
+		(stroke
+			(width 0)
+			(type default)
+		)
+	)
+	(wire
+		(pts
+			(xy 171.45 41.91) (xy 171.45 36.83)
 		)
 		(stroke
@@
 	(wire
 		(pts
-			(xy 173.99 113.03) (xy 173.99 91.44)
+			(xy 171.45 113.03) (xy 171.45 92.71)
 		)
 		(stroke
@@
 	(wire
 		(pts
-			(xy 128.27 34.29) (xy 134.62 34.29)
+			(xy 128.27 34.29) (xy 139.7 34.29)
 		)
 		(stroke
@@
 	(wire
 		(pts
-			(xy 162.56 41.91) (xy 173.99 41.91)
-		)
-		(stroke
-			(width 0)
-			(type default)
-		)
-	)
-	(wire
-		(pts
 			(xy 199.39 49.53) (xy 199.39 83.82)
 		)
@@
 	(wire
 		(pts
+			(xy 135.89 92.71) (xy 135.89 102.87)
+		)
+		(stroke
+			(width 0)
+			(type default)
+		)
+	)
+	(wire
+		(pts
 			(xy 179.07 160.02) (xy 179.07 157.48)
 		)
@@
 		)
 		(stroke
+			(width 0)
+			(type default)
+		)
+	)
+	(wire
+		(pts
+			(xy 135.89 102.87) (xy 139.7 102.87)
+		)
+		(stroke
