File: ip2366/ip2366/ip2366.kicad_sch (KiCad schematic)
At the start: 60 parts, among them CN1 XT30PW-M, Q1 RU3030M2-VB, SW1 K2-1112SW-A4SW-04, U1 IP2366 (I2C VERSION)

Commit message: aktueller stand
Parts:
- added R21: 0R, Resistor_SMD:R_0603_1608Metric_Pad0.98x0.95mm_HandSolder, symbol Device:R
Connections:
- net NTC: now also R21.1; no longer RNTC1.1
- net VBUS: now also Q1.1 (S), Q1.3 (S)
- new net: R21.2, RNTC1.1
Other:
- moved on the sheet: C21, RNTC1
Changed lines of the file:
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@@
 	)
 	(junction
+		(at 54.61 113.03)
+		(diameter 0)
+		(color 0 0 0 0)
+	)
+	(junction
 		(at 67.31 118.11)
 		(diameter 0)
@@
 	)
 	(junction
-		(at 226.06 67.31)
+		(at 229.87 68.58)
 		(diameter 0)
 		(color 0 0 0 0)
@@
 	)
 	(junction
-		(at 41.91 113.03)
-		(diameter 0)
-		(color 0 0 0 0)
-	)
-	(junction
 		(at 231.14 91.44)
 		(diameter 0)
@@
 	)
 	(junction
+		(at 41.91 113.03)
+		(diameter 0)
+		(color 0 0 0 0)
+	)
+	(junction
 		(at 156.21 99.06)
 		(diameter 0)
@@
 	)
 	(junction
-		(at 41.91 123.19)
-		(diameter 0)
-		(color 0 0 0 0)
-	)
-	(junction
 		(at 31.75 62.23)
 		(diameter 0)
@@
 		(color 0 0 0 0)
 	)
+	(junction
+		(at 41.91 123.19)
+		(diameter 0)
+		(color 0 0 0 0)
+	)
 	(no_connect
 		(at 31.75 41.91)
@@
 	(wire
 		(pts
+			(xy 41.91 113.03) (xy 48.26 113.03)
+		)
+		(stroke
+			(width 0)
+			(type default)
+		)
+	)
+	(wire
+		(pts
 			(xy 22.86 153.67) (xy 34.29 153.67)
 		)
@@
 	(wire
 		(pts
+			(xy 54.61 110.49) (xy 54.61 113.03)
+		)
+		(stroke
+			(width 0)
+			(type default)
+		)
+	)
+	(wire
+		(pts
 			(xy 105.41 76.2) (xy 105.41 96.52)
 		)
@@
 	(wire
 		(pts
-			(xy 215.9 63.5) (xy 215.9 71.12)
+			(xy 209.55 64.77) (xy 209.55 72.39)
 		)
 		(stroke
@@
 	(wire
 		(pts
-			(xy 237.49 151.13) (xy 243.84 151.13)
+			(xy 209.55 72.39) (xy 212.09 72.39)
 		)
 		(stroke
@@
 	(wire
 		(pts
-			(xy 41.91 123.19) (xy 48.26 123.19)
+			(xy 237.49 151.13) (xy 243.84 151.13)
 		)
 		(stroke
@@
 	(wire
 		(pts
-			(xy 217.17 63.5) (xy 215.9 63.5)
+			(xy 220.98 64.77) (xy 209.55 64.77)
 		)
 		(stroke
@@
 	(wire
 		(pts
-			(xy 41.91 113.03) (xy 48.26 113.03)
+			(xy 149.86 147.32) (xy 149.86 149.86)
 		)
 		(stroke
@@
 	(wire
 		(pts
-			(xy 149.86 147.32) (xy 149.86 149.86)
+			(xy 149.86 144.78) (xy 149.86 147.32)
 		)
 		(stroke
@@
 	(wire
 		(pts
-			(xy 149.86 144.78) (xy 149.86 147.32)
+			(xy 129.54 175.26) (xy 129.54 177.8)
 		)
 		(stroke
@@
 	(wire
 		(pts
-			(xy 129.54 175.26) (xy 129.54 177.8)
+			(xy 54.61 113.03) (xy 54.61 115.57)
 		)
 		(stroke
@@
 	(wire
 		(pts
-			(xy 226.06 71.12) (xy 226.06 67.31)
+			(xy 229.87 72.39) (xy 229.87 68.58)
 		)
 		(stroke
@@
 	(wire
 		(pts
-			(xy 226.06 63.5) (xy 224.79 63.5)
+			(xy 229.87 64.77) (xy 228.6 64.77)
 		)
 		(stroke
@@
 	(wire
 		(pts
-			(xy 226.06 67.31) (xy 226.06 63.5)
+			(xy 229.87 68.58) (xy 229.87 64.77)
 		)
 		(stroke
@@
 	(wire
 		(pts
+			(xy 41.91 123.19) (xy 48.26 123.19)
+		)
+		(stroke
+			(width 0)
+			(type default)
+		)
+	)
+	(wire
+		(pts
 			(xy 93.98 71.12) (xy 93.98 86.36)
 		)
@@
 	(global_label "NTC"
 		(shape input)
-		(at 215.9 67.31 180)
+		(at 209.55 67.31 180)
 		(fields_autoplaced yes)
 		(effects
@@
 		)
 		(property "Intersheetrefs" "${INTERSHEET_REFS}"
-			(at 209.3467 67.31 0)
+			(at 202.9967 67.31 0)
 			(effects
 				(font
@@
 	(symbol
 		(lib_id "Device:C")
-		(at 220.98 63.5 90)
+		(at 224.79 64.77 90)
 		(unit 1)
 		(exclude_from_sim no)
@@
 		(dnp no)
 		(property "Reference" "C21"
-			(at 222.504 58.928 90)
+			(at 226.314 60.198 90)
 			(effects
 				(font
@@
 		)
 		(property "Value" "100nF"
-			(at 223.52 57.15 90)
+			(at 227.33 58.42 90)
 			(effects
 				(font
@@
 		)
 		(property "Footprint" "Capacitor_SMD:C_0603_1608Metric_Pad1.08x0.95mm_HandSolder"
-			(at 224.79 62.5348 0)
+			(at 228.6 63.8048 0)
 			(effects
 				(font
@@
 		)
 		(property "Datasheet" "~"
-			(at 220.98 63.5 0)
+			(at 224.79 64.77 0)
 			(effects
 				(font
@@
 		)
 		(property "Description" "Unpolarized capacitor"
-			(at 220.98 63.5 0)
+			(at 224.79 64.77 0)
 			(effects
 				(font
@@
 	(symbol
 		(lib_id "easyeda2kicad:RC0603FR-0710KL")
-		(at 220.98 71.12 0)
+		(at 224.79 72.39 0)
 		(unit 1)
 		(exclude_from_sim no)
@@
 		(dnp no)
 		(property "Reference" "RNTC1"
-			(at 220.98 73.406 0)
+			(at 224.79 74.676 0)
 			(effects
 				(font
@@
 		)
 		(property "Value" "10k"
-			(at 220.98 75.184 0)
+			(at 224.79 76.454 0)
 			(effects
 				(font
@@
 		)
 		(property "Footprint" "easyeda2kicad:R0603"
-			(at 220.98 78.74 0)
+			(at 224.79 80.01 0)
 			(effects
 				(font
@@
 		)
 		(property "Datasheet" "https://lcsc.com/product-detail/Chip-Resistor-Surface-Mount_10KR-1_C98220.html"
-			(at 220.98 81.28 0)
+			(at 224.79 82.55 0)
 			(effects
 				(font
@@
 		)
 		(property "Description" ""
-			(at 220.98 71.12 0)
+			(at 224.79 72.39 0)
 			(effects
 				(font
@@
 		)
 		(property "LCSC Part" "C98220"
-			(at 220.98 83.82 0)
+			(at 224.79 85.09 0)
 			(effects
 				(font
@@
 	)
 	(symbol
+		(lib_id "Device:R")
+		(at 215.9 72.39 90)
+		(unit 1)
+		(exclude_from_sim no)
+		(in_bom yes)
+		(on_board yes)
+		(dnp no)
+		(property "Reference" "R21"
+			(at 215.9 70.104 90)
+			(effects
+				(font
+					(size 1.27 1.27)
+				)
+			)
+		)
+		(property "Value" "0R"
+			(at 215.9 72.39 90)
+			(effects
+				(font
+					(size 1.27 1.27)
+				)
+			)
+		)
+		(property "Footprint" "Resistor_SMD:R_0603_1608Metric_Pad0.98x0.95mm_HandSolder"
+			(at 215.9 74.168 90)
+			(effects
+				(font
+					(size 1.27 1.27)
+				)
+				(hide yes)
+			)
+		)
+		(property "Datasheet" "~"
+			(at 215.9 72.39 0)
+			(effects
+				(font
+					(size 1.27 1.27)
+				)
+				(hide yes)
+			)
+		)
+		(property "Description" "Resistor"
+			(at 215.9 72.39 0)
+			(effects
+				(font
+					(size 1.27 1.27)
+				)
+				(hide yes)
+			)
+		)
+		(pin "1"
+		)
+		(pin "2"
+		)
+		(instances
+			(project "ip2366"
+				(path "/2ca5f6a3-9021-4596-b870-f2bf74885223"
+					(reference "R21")
+					(unit 1)
+				)
+			)
+		)
+	)
+	(symbol
 		(lib_id "power:-BATT")
 		(at 153.67 113.03 90)
@@
 	(symbol
 		(lib_id "power:GND")
-		(at 226.06 67.31 90)
+		(at 229.87 68.58 90)
 		(unit 1)
 		(exclude_from_sim no)
@@
 		(fields_autoplaced yes)
 		(property "Reference" "#PWR015"
-			(at 232.41 67.31 0)
+			(at 236.22 68.58 0)
 			(effects
 				(font
@@
 		)
 		(property "Value" "GND"
-			(at 229.87 67.3099 90)
+			(at 233.68 68.5799 90)
 			(effects
 				(font
@@
 		)
 		(property "Footprint" ""
-			(at 226.06 67.31 0)
+			(at 229.87 68.58 0)
 			(effects
 				(font
@@
 		)
 		(property "Datasheet" ""
-			(at 226.06 67.31 0)
+			(at 229.87 68.58 0)
 			(effects
 				(font
@@
 		)
 		(property "Description" "Power symbol creates a global label with name \"GND\" , ground"
-			(at 226.06 67.31 0)
+			(at 229.87 68.58 0)
 			(effects
 				(font
