File: ledConnect/ledConnect.kicad_pcb (KiCad board)
At the start: 2 copper layers, 43.9 x 43.9 mm, 22 parts, among them Q1 AO4407A, SW1 SS-12M11G5, U1 MT30-M, U2 TPS565208DDCR

Commit message: testownbucklayout
Parts:
- moved C7 10.1 mm to (194.2, 138.0), turned to 0 degrees
- moved C6 9.89 mm to (195.0, 128.4), turned to 0 degrees
- moved C1 9.11 mm to (196.4, 148.7), turned to 0 degrees
- moved C4 8.66 mm to (192.9, 135.0), turned to -90 degrees
- moved C2 8.56 mm to (195.0, 130.4), turned to 0 degrees
- moved C5 8.26 mm to (194.2, 140.0), turned to 0 degrees
- moved C3 7.86 mm to (195.2, 132.2), turned to 0 degrees
- moved U2 7.42 mm to (195.2, 134.8), turned to 90 degrees
- moved L1 6.93 mm to (185.6, 139.7)
- moved TP5 6.87 mm to (200.0, 159.6)
- moved TP3 6.52 mm to (204.0, 159.6)
- moved TP2 5.80 mm to (200.0, 155.4)
- moved TP4 5.38 mm to (196.0, 155.4)
- moved TP1 5.18 mm to (196.0, 159.6)
- moved TP6 3.64 mm to (204.0, 155.4)
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Routing:
- net Net-(U2-SW): track 0.00 -> 3.48 mm
- added copper zone on B.Cu, net GND
- added copper zone on F.Cu, net Net-(U2-SW)
- added copper zone on F.Cu, net VDC
