File: balancingboardbyd/balancingboardbyd.kicad_sch (KiCad schematic)
At the start: 74 parts, among them CN1 XT30PW-M, CN2 WJ15EDGRC-3.81-4P, CN3 WJ15EDGRC-3.81-4P, Q1 KMBTA94, Q10 SI2302A-TP, Q11 IRFH5302TRPBF, Q2 SI2302A-TP, Q3 SI2302A-TP, Q4 SI2302A-TP, Q5 SI2302A-TP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

Commit message: next step
Parts:
- added BT1, BT2, BT3: BH-18650-B1BA007, easyeda2kicad:BAT-SMD_BH-18650-B1BA007, symbol easyeda2kicad:BH-18650-B1BA007
- added U4, U5, U6, U7, U8, U9: BH-21700-B1BJ001, easyeda2kicad:BAT-SMD_L82.5.5-W25-BH-21700-B1BJ001, symbol easyeda2kicad:BH-21700-B1BJ001
Connections:
- net BAT+ is gone; now on net B8: CN1.2 (+), U3.1
- net B3: now also BT3.2, BT3.4, U8.2, U9.1
- net B4: now also BT2.3, BT3.1, U7.2, U8.1
- net B5: now also BT2.2, BT2.4, U6.2, U7.1
- net B6: now also BT1.3, BT2.1, U5.2, U6.1
- net B7: now also BT1.2, BT1.4, U4.2, U5.1
- net B8: now also BT1.1, U4.1
- net GND: now also BT3.3, U9.2
Other:
- note added: "+"
- note added: "-"
- moved on the sheet: CN2, CN3

Commit message: balancing board route
Parts:
- removed C11, C12: 0.1uF, Capacitor_SMD:C_0603_1608Metric_Pad1.08x0.95mm_HandSolder, symbol Device:C
Connections:
- net at RP1.1, U1.12 (DO): now also Q1.2 (E); no longer Q1.3 (C)
- net at Q6.2 (E): now also Q1.3 (C); no longer Q1.2 (E)
Changed lines of the file:
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@@
 	)
 	(junction
-		(at 200.66 191.77)
-		(diameter 0)
-		(color 0 0 0 0)
-	)
-	(junction
 		(at 73.66 133.35)
 		(diameter 0)
@@
 	)
 	(junction
-		(at 190.5 191.77)
-		(diameter 0)
-		(color 0 0 0 0)
-	)
-	(junction
 		(at 106.68 196.85)
 		(diameter 0)
@@
 	(wire
 		(pts
-			(xy 190.5 191.77) (xy 200.66 191.77)
-		)
-		(stroke
-			(width 0)
-			(type default)
-		)
-	)
-	(wire
-		(pts
 			(xy 214.63 87.63) (xy 224.79 87.63)
 		)
@@
 	(wire
 		(pts
-			(xy 180.34 191.77) (xy 190.5 191.77)
+			(xy 180.34 191.77) (xy 214.63 191.77)
 		)
 		(stroke
@@
 	(wire
 		(pts
-			(xy 200.66 191.77) (xy 214.63 191.77)
-		)
-		(stroke
-			(width 0)
-			(type default)
-		)
-	)
-	(wire
-		(pts
 			(xy 184.15 71.12) (xy 161.29 71.12)
 		)
@@
 		)
 	)
-	(label "VC2"
-		(at 190.5 184.15 0)
-		(effects
-			(font
-				(size 1.27 1.27)
-			)
-			(justify left bottom)
-		)
-	)
 	(label "VC8"
 		(at 157.48 50.8 0)
@@
 		)
 	)
-	(label "VC1"
-		(at 200.66 184.15 0)
-		(effects
-			(font
-				(size 1.27 1.27)
-			)
-			(justify left bottom)
-		)
-	)
 	(label "VC5"
 		(at 160.02 184.15 0)
@@
 	(symbol
 		(lib_id "Device:C")
-		(at 190.5 187.96 180)
-		(unit 1)
-		(exclude_from_sim no)
-		(in_bom yes)
-		(on_board yes)
-		(dnp no)
-		(property "Reference" "C11"
-			(at 194.818 186.944 0)
-			(effects
-				(font
-					(size 1.27 1.27)
-				)
-			)
-		)
-		(property "Value" "0.1uF"
-			(at 195.58 188.722 0)
-			(effects
-				(font
-					(size 1.27 1.27)
-				)
-			)
-		)
-		(property "Footprint" "Capacitor_SMD:C_0603_1608Metric_Pad1.08x0.95mm_HandSolder"
-			(at 189.5348 184.15 0)
-			(effects
-				(font
-					(size 1.27 1.27)
-				)
-				(hide yes)
-			)
-		)
-		(property "Datasheet" "~"
-			(at 190.5 187.96 0)
-			(effects
-				(font
-					(size 1.27 1.27)
-				)
-				(hide yes)
-			)
-		)
-		(property "Description" "Unpolarized capacitor"
-			(at 190.5 187.96 0)
-			(effects
-				(font
-					(size 1.27 1.27)
-				)
-				(hide yes)
-			)
-		)
-		(pin "1"
-		)
-		(pin "2"
-		)
-		(instances
-			(project "balancingboardbyd"
-				(path "/ad801e52-4300-4542-ba97-19e7ee181034"
-					(reference "C11")
-					(unit 1)
-				)
-			)
-		)
-	)
-	(symbol
-		(lib_id "Device:C")
 		(at 85.09 138.43 90)
 		(unit 1)
@@
 		(lib_id "easyeda2kicad:KMBTA94")
 		(at 111.76 100.33 0)
+		(mirror x)
 		(unit 1)
 		(exclude_from_sim no)
@@
 		(on_board yes)
 		(dnp no)
-		(fields_autoplaced yes)
 		(property "Reference" "Q1"
 			(at 113.03 99.0599 0)
@@
 		)
 		(property "Footprint" "easyeda2kicad:SOT-23-3_L2.9-W1.3-P1.90-LS2.4-BR"
-			(at 111.76 113.03 0)
+			(at 111.76 87.63 0)
 			(effects
 				(font
@@
 		)
 		(property "Datasheet" "https://lcsc.com/product-detail/New-Arrivals_KEXIN-KMBTA94_C489166.html"
-			(at 111.76 115.57 0)
+			(at 111.76 85.09 0)
 			(effects
 				(font
@@
 		)
 		(property "LCSC Part" "C489166"
-			(at 111.76 118.11 0)
+			(at 111.76 82.55 0)
 			(effects
 				(font
@@
 		)
 		(instances
-			(project ""
+			(project "balancingboardbyd"
 				(path "/ad801e52-4300-4542-ba97-19e7ee181034"
 					(reference "Q1")
@@
 					(unit 1)
 				)
-			)
-		)
-	)
-	(symbol
-		(lib_id "Device:C")
-		(at 200.66 187.96 180)
-		(unit 1)
-		(exclude_from_sim no)
-		(in_bom yes)
-		(on_board yes)
-		(dnp no)
-		(property "Reference" "C12"
-			(at 204.978 186.944 0)
-			(effects
-				(font
-					(size 1.27 1.27)
-				)
-			)
-		)
-		(property "Value" "0.1uF"
-			(at 205.74 188.722 0)
-			(effects
-				(font
-					(size 1.27 1.27)
-				)
-			)
-		)
-		(property "Footprint" "Capacitor_SMD:C_0603_1608Metric_Pad1.08x0.95mm_HandSolder"
-			(at 199.6948 184.15 0)
-			(effects
-				(font
-					(size 1.27 1.27)
-				)
-				(hide yes)
-			)
-		)
-		(property "Datasheet" "~"
-			(at 200.66 187.96 0)
-			(effects
-				(font
-					(size 1.27 1.27)
-				)
-				(hide yes)
-			)
-		)
-		(property "Description" "Unpolarized capacitor"
-			(at 200.66 187.96 0)
-			(effects
-				(font
-					(size 1.27 1.27)
-				)
-				(hide yes)
-			)
-		)
-		(pin "1"
-		)
-		(pin "2"
-		)
-		(instances
-			(project "balancingboardbyd"
-				(path "/ad801e52-4300-4542-ba97-19e7ee181034"
-					(reference "C12")
-					(unit 1)
-				)

Commit message: kurz vor bestellung
Parts:
- removed CN2, CN3: WJ15EDGRC-3.81-4P, easyeda2kicad:CONN-TH_WJ15EDGRC-3.81-4P, symbol easyeda2kicad:WJ15EDGRC-3.81-4P
- added CN4, CN5: WJ15EDGVC-3.81-4P, easyeda2kicad:CONN-TH_4P-P3.81_WJ2EDGVC-3.81-4P, symbol easyeda2kicad:WJ15EDGVC-3.81-4P
Connections:
- net B3: now also CN5.2
- net B4: now also CN5.3
- net B5: now also CN5.4
- net B6: now also CN4.1
- net B7: now also CN4.2
- net B8: now also CN4.3
- net GND: now also CN5.1
Changed lines of the file:
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@@
 	)
 	(symbol
-		(lib_id "easyeda2kicad:WJ15EDGRC-3.81-4P")
-		(at 288.29 135.89 0)
-		(mirror x)
-		(unit 1)
-		(exclude_from_sim no)
-		(in_bom yes)
-		(on_board yes)
-		(dnp no)
-		(property "Reference" "CN3"
-			(at 294.64 136.9051 0)
-			(effects
-				(font
-					(size 1.27 1.27)
-				)
-				(justify left)
-			)
-		)
-		(property "Value" "WJ15EDGRC-3.81-4P"
-			(at 294.64 134.3651 0)
-			(effects
-				(font
-					(size 1.27 1.27)
-				)
-				(justify left)
-			)
-		)
-		(property "Footprint" "easyeda2kicad:CONN-TH_WJ15EDGRC-3.81-4P"
-			(at 288.29 124.46 0)
-			(effects
-				(font
-					(size 1.27 1.27)
-				)
-				(hide yes)
-			)
-		)
-		(property "Datasheet" "https://lcsc.com/product-detail/15EDG-Connectors_WJ15EDGRC-3-81-4P_C7245.html"
-			(at 288.29 121.92 0)
-			(effects
-				(font
-					(size 1.27 1.27)
-				)
-				(hide yes)
-			)
-		)
-		(property "Description" ""
-			(at 288.29 135.89 0)
-			(effects
-				(font
-					(size 1.27 1.27)
-				)
-				(hide yes)
-			)
-		)
-		(property "LCSC Part" "C7245"
-			(at 288.29 119.38 0)
-			(effects
-				(font
-					(size 1.27 1.27)
-				)
-				(hide yes)
-			)
-		)
-		(pin "1"
-		)
-		(pin "2"
-		)
-		(pin "3"
-		)
-		(pin "4"
-		)
-		(instances
-			(project "balancingboardbyd"
-				(path "/ad801e52-4300-4542-ba97-19e7ee181034"
-					(reference "CN3")
-					(unit 1)
-				)
-			)
-		)
-	)
-	(symbol
 		(lib_id "easyeda2kicad:BH-18650-B1BA007")
 		(at 331.47 60.96 0)
@@
 	)
 	(symbol
-		(lib_id "Device:C")
-		(at 105.41 130.81 90)
+		(lib_id "easyeda2kicad:WJ15EDGVC-3.81-4P")
+		(at 289.56 120.65 0)
+		(mirror x)
 		(unit 1)
 		(exclude_from_sim no)
@@
 		(on_board yes)
 		(dnp no)
-		(property "Reference" "C14"
-			(at 105.41 134.366 90)
+		(property "Reference" "CN4"
+			(at 294.64 122.9351 0)
+			(effects
+				(font
+					(size 1.27 1.27)
+				)
+				(justify left)
+			)
+		)
+		(property "Value" "WJ15EDGVC-3.81-4P"
+			(at 294.64 120.3951 0)
 			(effects
 				(font
 					(size 1.27 1.27)
 				)
+				(justify left)
 			)
 		)
-		(property "Value" "10nF"
-			(at 105.41 135.89 90)
+		(property "Footprint" "easyeda2kicad:CONN-TH_4P-P3.81_WJ2EDGVC-3.81-4P"
+			(at 289.56 110.49 0)
 			(effects
 				(font
 					(size 1.27 1.27)
 				)
+				(hide yes)
 			)
 		)
-		(property "Footprint" "Capacitor_SMD:C_0603_1608Metric_Pad1.08x0.95mm_HandSolder"
-			(at 109.22 129.8448 0)
+		(property "Datasheet" "https://lcsc.com/product-detail/15EDG-Connectors_WJ15EDGVC-3-81-4P_C8410.html"
+			(at 289.56 107.95 0)
 			(effects
 				(font
@@
 			)
 		)
-		(property "Datasheet" "~"
-			(at 105.41 130.81 0)
+		(property "Description" ""
+			(at 289.56 120.65 0)
 			(effects
 				(font
@@
 			)
 		)
-		(property "Description" "Unpolarized capacitor"
-			(at 105.41 130.81 0)
+		(property "LCSC Part" "C8410"
+			(at 289.56 105.41 0)
 			(effects
 				(font
@@
 		(pin "1"
 		)
+		(pin "3"
+		)
+		(pin "4"
+		)
 		(pin "2"
 		)
 		(instances
-			(project "balancingboardbyd"
+			(project ""
 				(path "/ad801e52-4300-4542-ba97-19e7ee181034"
-					(reference "C14")
+					(reference "CN4")
 					(unit 1)
 				)
@@
 	)
 	(symbol
-		(lib_id "easyeda2kicad:WJ15EDGRC-3.81-4P")
-		(at 288.29 121.92 0)
-		(mirror x)
+		(lib_id "Device:C")
+		(at 105.41 130.81 90)
 		(unit 1)
 		(exclude_from_sim no)
@@
 		(on_board yes)
 		(dnp no)
-		(property "Reference" "CN2"
-			(at 294.64 122.9351 0)
-			(effects
-				(font
-					(size 1.27 1.27)
-				)
-				(justify left)
-			)
-		)
-		(property "Value" "WJ15EDGRC-3.81-4P"
-			(at 294.64 120.3951 0)
+		(property "Reference" "C14"
+			(at 105.41 134.366 90)
 			(effects
 				(font
 					(size 1.27 1.27)
 				)
-				(justify left)
 			)
 		)
-		(property "Footprint" "easyeda2kicad:CONN-TH_WJ15EDGRC-3.81-4P"
-			(at 288.29 110.49 0)
+		(property "Value" "10nF"
+			(at 105.41 135.89 90)
 			(effects
 				(font
 					(size 1.27 1.27)
 				)
-				(hide yes)
 			)
 		)
-		(property "Datasheet" "https://lcsc.com/product-detail/15EDG-Connectors_WJ15EDGRC-3-81-4P_C7245.html"
-			(at 288.29 107.95 0)
+		(property "Footprint" "Capacitor_SMD:C_0603_1608Metric_Pad1.08x0.95mm_HandSolder"
+			(at 109.22 129.8448 0)
 			(effects
 				(font
@@
 			)
 		)
-		(property "Description" ""
-			(at 288.29 121.92 0)
+		(property "Datasheet" "~"
+			(at 105.41 130.81 0)
 			(effects
 				(font
@@
 			)
 		)
-		(property "LCSC Part" "C7245"
-			(at 288.29 105.41 0)
+		(property "Description" "Unpolarized capacitor"
+			(at 105.41 130.81 0)
 			(effects
 				(font
@@
 		(pin "2"
 		)
-		(pin "3"
-		)
-		(pin "4"
-		)
 		(instances
-			(project ""
+			(project "balancingboardbyd"
 				(path "/ad801e52-4300-4542-ba97-19e7ee181034"
-					(reference "CN2")
+					(reference "C14")
 					(unit 1)
 				)
@@
 					(unit 1)
 				)
+			)
+		)
+	)
+	(symbol
+		(lib_id "easyeda2kicad:WJ15EDGVC-3.81-4P")
+		(at 289.56 134.62 0)
+		(mirror x)
+		(unit 1)
+		(exclude_from_sim no)
+		(in_bom yes)
+		(on_board yes)
+		(dnp no)
+		(property "Reference" "CN5"
+			(at 294.64 136.9051 0)
+			(effects
+				(font
+					(size 1.27 1.27)
+				)
+				(justify left)
+			)
+		)
+		(property "Value" "WJ15EDGVC-3.81-4P"
+			(at 294.64 134.3651 0)
+			(effects
+				(font
+					(size 1.27 1.27)
+				)
+				(justify left)
+			)
+		)
+		(property "Footprint" "easyeda2kicad:CONN-TH_4P-P3.81_WJ2EDGVC-3.81-4P"
+			(at 289.56 124.46 0)
+			(effects
+				(font
+					(size 1.27 1.27)
+				)
+				(hide yes)
+			)
+		)
+		(property "Datasheet" "https://lcsc.com/product-detail/15EDG-Connectors_WJ15EDGVC-3-81-4P_C8410.html"
+			(at 289.56 121.92 0)
+			(effects
+				(font
+					(size 1.27 1.27)
+				)
+				(hide yes)
+			)
+		)
+		(property "Description" ""
+			(at 289.56 134.62 0)
+			(effects
+				(font
+					(size 1.27 1.27)
+				)
+				(hide yes)
+			)
+		)
+		(property "LCSC Part" "C8410"
+			(at 289.56 119.38 0)
+			(effects
+				(font
+					(size 1.27 1.27)
+				)
+				(hide yes)
+			)
+		)
+		(pin "1"
+		)
+		(pin "3"
+		)
+		(pin "4"
+		)
+		(pin "2"
+		)
+		(instances
+			(project "balancingboardbyd"
+				(path "/ad801e52-4300-4542-ba97-19e7ee181034"
+					(reference "CN5")
+					(unit 1)
+				)
