File: ledBrain/ledBrain.kicad_pcb (KiCad board)
At the start: 2 copper layers, 34.2 x 70.7 mm, 26 parts, among them CN1 XT30PW-M, SW2 K2-1112SW-A4SW-04, SW3 K2-1112SW-A4SW-04, U1 QuinLED-ESP32, U2 MT30-F, U3 CH224A, U4 LM2940S-5.0, U5 SN74AHCT32QPWRQ1

Commit message: bestelle teile
Routing:
- net GND: track 0.00 -> 13.2 mm, vias 0 -> 108
- net +5V: track 78.9 -> 85.9 mm
- net VBUS: vias 0 -> 94

Commit message: kurz vor bestellung
Other:
- board text added: "Janek"
- board text added: "github.com/janekc"
