File: ledBrain/ledBrain.kicad_pcb (KiCad board)
At the start: 4 copper layers, 34.2 x 70.7 mm, 44 parts, among them CN1 XT30PW-M, SW1 EC11E09244BS, SW2 K2-1112SW-A4SW-04, U1 QuinLED-ESP32, U10 HS96L03W2C03, U2 MSM261DGT003, U3 CH224A, U4 ME3116, U5 SN74AHCT32QPWRQ1, U7 T34069, U8 T34069, U9 T34069

Commit message: updates
Other:
- board text added: "DATA"
- board text added: "GND"
- board text added: "VDD"
Changed lines of the file:
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@@
 		(layer "Edge.Cuts")
+	)
+	(gr_text "VDD"
+		(at 154.2 45.13 0)
+		(layer "F.SilkS")
+		(effects
+			(font
+				(face "Inconsolata LGC Nerd Font")
+				(size 1 1)
+				(thickness 0.2)
+				(bold yes)
+			)
+			(justify left bottom)
+		)
+		(render_cache "VDD" 0
+			(polygon
+				(pts
+					(xy 154.22595 43.949811) (xy 154.388677 43.949811) (xy 154.632004 44.67967) (xy 154.861714 43.951765)
+					(xy 155.018946 43.951765) (xy 154.666198 44.967815) (xy 154.584193 44.967815)
+				)
+			)
+			(polygon
+				(pts
+					(xy 155.456111 43.951951) (xy 155.522964 43.963209) (xy 155.577032 43.980366) (xy 155.620455 44.002568)
+					(xy 155.666747 44.036488) (xy 155.706816 44.077311) (xy 155.741063 44.125654) (xy 155.769565 44.182452)
+					(xy 155.796388 44.262749) (xy 155.813055 44.351874) (xy 155.818841 44.451181) (xy 155.811651 44.559265)
+					(xy 155.791046 44.654615) (xy 155.757964 44.739143) (xy 155.723363 44.797913) (xy 155.682723 44.846838)
+					(xy 155.635838 44.886979) (xy 155.582109 44.918967) (xy 155.524862 44.940346) (xy 155.450071 44.954677)
+					(xy 155.353558 44.96) (xy 155.115422 44.96) (xy 155.115422 44.827131) (xy 155.263921 44.827131)
+					(xy 155.346659 44.827131) (xy 155.424253 44.821938) (xy 155.482623 44.808076) (xy 155.525933 44.787442)
+					(xy 155.572311 44.750319) (xy 155.609372 44.702003) (xy 155.63748 44.640452) (xy 155.655828 44.562646)
+					(xy 155.662526 44.464797) (xy 155.656576 44.364468) (xy 155.640304 44.284384) (xy 155.615552 44.220922)
+					(xy 155.583362 44.171054) (xy 155.543885 44.132505) (xy 155.503922 44.10732) (xy 155.464567 44.093548)
+					(xy 155.421737 44.087061) (xy 155.366015 44.084633) (xy 155.263921 44.084633) (xy 155.263921 44.827131)
+					(xy 155.115422 44.827131) (xy 155.115422 43.947857) (xy 155.374014 43.947857)
+				)
+			)
+			(polygon
+				(pts
+					(xy 156.293375 43.951951) (xy 156.360229 43.963209) (xy 156.414297 43.980366) (xy 156.457719 44.002568)
+					(xy 156.504012 44.036488) (xy 156.54408 44.077311) (xy 156.578328 44.125654) (xy 156.60683 44.182452)
+					(xy 156.633652 44.262749) (xy 156.650319 44.351874) (xy 156.656106 44.451181) (xy 156.648915 44.559265)
+					(xy 156.628311 44.654615) (xy 156.595228 44.739143) (xy 156.560627 44.797913) (xy 156.519988 44.846838)
+					(xy 156.473102 44.886979) (xy 156.419373 44.918967) (xy 156.362126 44.940346) (xy 156.287336 44.954677)
+					(xy 156.190823 44.96) (xy 155.952686 44.96) (xy 155.952686 44.827131) (xy 156.101186 44.827131)
+					(xy 156.183923 44.827131) (xy 156.261517 44.821938) (xy 156.319887 44.808076) (xy 156.363197 44.787442)
+					(xy 156.409575 44.750319) (xy 156.446637 44.702003) (xy 156.474744 44.640452) (xy 156.493092 44.562646)
+					(xy 156.49979 44.464797) (xy 156.49384 44.364468) (xy 156.477569 44.284384) (xy 156.452817 44.220922)
+					(xy 156.420626 44.171054) (xy 156.381149 44.132505) (xy 156.341186 44.10732) (xy 156.301831 44.093548)
+					(xy 156.259002 44.087061) (xy 156.203279 44.084633) (xy 156.101186 44.084633) (xy 156.101186 44.827131)
+					(xy 155.952686 44.827131) (xy 155.952686 43.947857) (xy 156.211278 43.947857)
+				)
+			)
+		)
+	)
+	(gr_text "DATA\n"
+		(at 162.24 45.1 0)
+		(layer "F.SilkS")
+		(effects
+			(font
+				(face "Inconsolata LGC Nerd Font")
+				(size 1 1)
+				(thickness 0.2)
+				(bold yes)
+			)
+			(justify left bottom)
+		)
+		(render_cache "DATA\n" 0
+			(polygon
+				(pts
+					(xy 162.658847 43.921951) (xy 162.7257 43.933209) (xy 162.779768 43.950366) (xy 162.82319 43.972568)
+					(xy 162.869483 44.006488) (xy 162.909552 44.047311) (xy 162.943799 44.095654) (xy 162.972301 44.152452)
+					(xy 162.999123 44.232749) (xy 163.01579 44.321874) (xy 163.021577 44.421181) (xy 163.014386 44.529265)
+					(xy 162.993782 44.624615) (xy 162.960699 44.709143) (xy 162.926098 44.767913) (xy 162.885459 44.816838)
+					(xy 162.838573 44.856979) (xy 162.784844 44.888967) (xy 162.727597 44.910346) (xy 162.652807 44.924677)
+					(xy 162.556294 44.93) (xy 162.318157 44.93) (xy 162.318157 44.797131) (xy 162.466657 44.797131)
+					(xy 162.549394 44.797131) (xy 162.626988 44.791938) (xy 162.685358 44.778076) (xy 162.728668 44.757442)
+					(xy 162.775046 44.720319) (xy 162.812108 44.672003) (xy 162.840215 44.610452) (xy 162.858563 44.532646)
+					(xy 162.865261 44.434797) (xy 162.859311 44.334468) (xy 162.84304 44.254384) (xy 162.818288 44.190922)
+					(xy 162.786097 44.141054) (xy 162.74662 44.102505) (xy 162.706657 44.07732) (xy 162.667302 44.063548)
+					(xy 162.624473 44.057061) (xy 162.56875 44.054633) (xy 162.466657 44.054633) (xy 162.466657 44.797131)
+					(xy 162.318157 44.797131) (xy 162.318157 43.917857) (xy 162.576749 43.917857)
+				)
+			)
+			(polygon
+				(pts
+					(xy 163.905797 44.93061) (xy 163.74307 44.93061) (xy 163.630963 44.656448) (xy 163.339764 44.656448)
+					(xy 163.242677 44.931953) (xy 163.085446 44.931953) (xy 163.231533 44.527487) (xy 163.376706 44.527487)
+					(xy 163.58993 44.527487) (xy 163.479227 44.226458) (xy 163.376706 44.527487) (xy 163.231533 44.527487)
+					(xy 163.457367 43.902226) (xy 163.499743 43.902226)
+				)
+			)
+			(polygon
+				(pts
+					(xy 163.957515 43.917857) (xy 164.700013 43.917857) (xy 164.700013 44.062449) (xy 164.399106 44.062449)
+					(xy 164.399106 44.931953) (xy 164.242791 44.931953) (xy 164.242791 44.062449) (xy 163.957515 44.062449)
+				)
+			)
+			(polygon
+				(pts
+					(xy 165.580326 44.93061) (xy 165.417599 44.93061) (xy 165.305491 44.656448) (xy 165.014293 44.656448)
+					(xy 164.917206 44.931953) (xy 164.759975 44.931953) (xy 164.906062 44.527487) (xy 165.051235 44.527487)
+					(xy 165.264459 44.527487) (xy 165.153756 44.226458) (xy 165.051235 44.527487) (xy 164.906062 44.527487)
+					(xy 165.131896 43.902226) (xy 165.174272 43.902226)
+				)
+			)
+		)
+	)
+	(gr_text "GND"
+		(at 171.2 45.1 0)
+		(layer "F.SilkS")
+		(effects
+			(font
+				(face "Inconsolata LGC Nerd Font")
+				(size 1 1)
+				(thickness 0.2)
+				(bold yes)
+			)
+			(justify left bottom)
+		)
+		(render_cache "GND" 0
+			(polygon
+				(pts
+					(xy 171.661252 43.910041) (xy 171.726759 43.91543) (xy 171.786109 43.931125) (xy 171.84045 43.956929)
+					(xy 171.890653 43.993319) (xy 171.937253 44.041419) (xy 171.980416 44.102932) (xy 171.878995 44.20875)
+					(xy 171.853166 44.188845) (xy 171.835458 44.157887) (xy 171.808014 44.11558) (xy 171.768169 44.08095)
+					(xy 171.736612 44.064321) (xy 171.70173 44.054208) (xy 171.662718 44.050725) (xy 171.622805 44.054258)
+					(xy 171.584031 44.06487) (xy 171.545847 44.082904) (xy 171.511399 44.107208) (xy 171.481112 44.138185)
+					(xy 171.454745 44.176632) (xy 171.42992 44.235296) (xy 171.413302 44.312666) (xy 171.407117 44.413487)
+					(xy 171.413961 44.523248) (xy 171.432528 44.609156) (xy 171.460576 44.675793) (xy 171.496938 44.726912)
+					(xy 171.535589 44.761517) (xy 171.577188 44.785574) (xy 171.622463 44.800016) (xy 171.672487 44.804947)
+					(xy 171.726565 44.799779) (xy 171.779816 44.784132) (xy 171.833077 44.757259) (xy 171.833077 44.566566)
+					(xy 171.65075 44.566566) (xy 171.65075 44.425882) (xy 171.977669 44.425882) (xy 171.977669 44.834989)
+					(xy 171.928806 44.868456) (xy 171.84877 44.908079) (xy 171.790025 44.928784) (xy 171.727743 44.941354)
+					(xy 171.661252 44.945631) (xy 171.603173 44.941545) (xy 171.546031 44.929267) (xy 171.490888 44.907773)
+					(xy 171.435572 44.874617) (xy 171.385274 44.83206) (xy 171.340806 44.779668) (xy 171.305128 44.717603)
+					(xy 171.275348 44.634832) (xy 171.257221 44.543654) (xy 171.250802 44.437362) (xy 171.254288 44.354782)
+					(xy 171.264261 44.281123) (xy 171.280111 44.215406) (xy 171.302851 44.151358) (xy 171.327535 44.101106)
+					(xy 171.35375 44.062388) (xy 171.401719 44.011605) (xy 171.456027 43.970858) (xy 171.513865 43.939687)
+					(xy 171.563066 43.922376) (xy 171.61234 43.913102)
+				)
+			)
+			(polygon
+				(pts
+					(xy 172.111514 44.926092) (xy 172.111514 43.917857) (xy 172.255678 43.917857) (xy 172.646894 44.606866)
+					(xy 172.646894 43.917857) (xy 172.807545 43.917857) (xy 172.810903 43.946556) (xy 172.803393 43.965912)
+					(xy 172.799302 43.97788) (xy 172.799302 44.93) (xy 172.675715 44.93) (xy 172.263921 44.192081)
+					(xy 172.263921 44.926092)
+				)
+			)
+			(polygon
+				(pts
+					(xy 173.293375 43.921951) (xy 173.360229 43.933209) (xy 173.414297 43.950366) (xy 173.457719 43.972568)
+					(xy 173.504012 44.006488) (xy 173.54408 44.047311) (xy 173.578328 44.095654) (xy 173.60683 44.152452)
+					(xy 173.633652 44.232749) (xy 173.650319 44.321874) (xy 173.656106 44.421181) (xy 173.648915 44.529265)
+					(xy 173.628311 44.624615) (xy 173.595228 44.709143) (xy 173.560627 44.767913) (xy 173.519988 44.816838)
+					(xy 173.473102 44.856979) (xy 173.419373 44.888967) (xy 173.362126 44.910346) (xy 173.287336 44.924677)
+					(xy 173.190823 44.93) (xy 172.952686 44.93) (xy 172.952686 44.797131) (xy 173.101186 44.797131)
+					(xy 173.183923 44.797131) (xy 173.261517 44.791938) (xy 173.319887 44.778076) (xy 173.363197 44.757442)
+					(xy 173.409575 44.720319) (xy 173.446637 44.672003) (xy 173.474744 44.610452) (xy 173.493092 44.532646)
+					(xy 173.49979 44.434797) (xy 173.49384 44.334468) (xy 173.477569 44.254384) (xy 173.452817 44.190922)
+					(xy 173.420626 44.141054) (xy 173.381149 44.102505) (xy 173.341186 44.07732) (xy 173.301831 44.063548)
+					(xy 173.259002 44.057061) (xy 173.203279 44.054633) (xy 173.101186 44.054633) (xy 173.101186 44.797131)
+					(xy 172.952686 44.797131) (xy 172.952686 43.917857) (xy 173.211278 43.917857)
+				)
+			)
+		)
 	)
 	(gr_text "github.com/janekc"

Commit message: update stuff a little bit
Parts:
- added J1: Conn_01x06_Pin, Connector_PinHeader_2.54mm:PinHeader_1x06_P2.54mm_Vertical, F.Cu at (140.0, 62.4)
