File: ledConnectLongVersion/ledConnectLongVersion.kicad_pcb (KiCad board)
At the start: 4 copper layers, 21 x 60.9 mm, 18 parts, among them Q1 AO4407A, U2 LM61495RPHR

Commit message: update
Parts:
- added TP7: VIN_Connect, TestPoint:TestPoint_Plated_Hole_D3.0mm, F.Cu at (151.5, 111.5)
- added TP8: GND_Connect, TestPoint:TestPoint_Plated_Hole_D3.0mm, F.Cu at (137.5, 111.5)
- added TP9: VDC_Connect, TestPoint:TestPoint_Plated_Hole_D3.0mm, F.Cu at (144.5, 111.5)
- moved C1 55.2 mm to (140.0, 106.5), turned to 180 degrees
- moved R2 23.3 mm to (147.4, 92.0), turned to -90 degrees
- moved R1 20.2 mm to (149.0, 92.0), turned to 90 degrees
- moved Q1 13.6 mm to (152.2, 92.0), turned to 180 degrees
- moved Cout1 0.91 mm to (148.2, 101.9)
- moved L1 0.33 mm to (140.4, 96.2)
Connections:
- Cin1 pad 1: Net-(U2-VIN1) -> VIN2
- Cin2 pad 1: Net-(U2-VIN1) -> VIN2
- Cinx1 pad 1: Net-(U2-VIN1) -> VIN2
- Cinx2 pad 1: Net-(U2-VIN1) -> VIN2
- Q1 pad 1: Net-(U2-VIN1) -> VIN2
- Q1 pad 2: Net-(U2-VIN1) -> VIN2
- Q1 pad 3: Net-(U2-VIN1) -> VIN2
- U2 pad 14: Net-(U2-VIN1) -> VIN2
- U2 pad 2: Net-(U2-VIN1) -> VIN2
Routing:
- net VDC: track 12.5 -> 98.7 mm
- net VIN2: track 1.12 -> 2.45 mm
- net Net-(U2-VIN1): track 1.33 -> 0.00 mm
- net GND: vias 0 -> 24
- added copper zone on F.Cu, net VDC
- removed copper zone on F.Cu, net Net-(U2-VIN1)
Other:
- board size 21 x 60.9 mm -> 21 x 42 mm
- board text added: "GND"
- board text added: "Vin"
- board text added: "Vout"
