File: ledConnectLongVersion/ledConnectLongVersion.kicad_sch (KiCad schematic)
At the start: 21 parts, among them Q1 AO4407A, U2 LM61495RPHR

Commit message: update
Parts:
- TP7, TP8, TP9: footprint (none) -> TestPoint:TestPoint_Plated_Hole_D3.0mm
Connections:
- net VIN2: now also Cin1.1, Cin2.1, Cinx1.1, Cinx2.1, Q1.1 (S), Q1.2 (S), Q1.3 (S), U2.14 (VIN1), U2.2 (VIN2)
Changed lines of the file:
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@@
+		)
+	)
+	(label "VIN2"
+		(at 115.57 81.28 0)
+		(effects
+			(font
+				(size 1.27 1.27)
+			)
+			(justify left bottom)
 		)
 	)
@@
 			)
 		)
-		(property "Footprint" ""
+		(property "Footprint" "TestPoint:TestPoint_Plated_Hole_D3.0mm"
 			(at 120.65 127 0)
 			(hide yes)
@@
 			)
 		)
-		(property "Footprint" ""
+		(property "Footprint" "TestPoint:TestPoint_Plated_Hole_D3.0mm"
 			(at 120.65 151.13 0)
 			(hide yes)
@@
 			)
 		)
-		(property "Footprint" ""
+		(property "Footprint" "TestPoint:TestPoint_Plated_Hole_D3.0mm"
 			(at 120.65 138.43 0)
 			(hide yes)
