File: QuinledPoEHat/QuinledPoEHat.kicad_pcb (KiCad board)
At the start: 4 copper layers, 34.2 x 70.7 mm, 2 parts

Commit message: update lcsc bestellt
Parts:
- added C1: 100nF, Capacitor_SMD:C_0603_1608Metric_Pad1.08x0.95mm_HandSolder, F.Cu at (219.9, 41.1)
- added C10: 10nF, Capacitor_SMD:C_0603_1608Metric_Pad1.08x0.95mm_HandSolder, F.Cu at (219.9, 63.6)
- added C11: 10nF, Capacitor_SMD:C_0603_1608Metric_Pad1.08x0.95mm_HandSolder, F.Cu at (219.9, 66.2)
- added C12: 10nF, Capacitor_SMD:C_0603_1608Metric_Pad1.08x0.95mm_HandSolder, F.Cu at (224.2, 41.1)
- added C13: 10nF, Capacitor_SMD:C_0603_1608Metric_Pad1.08x0.95mm_HandSolder, F.Cu at (224.2, 43.6)
- added C14: 100nF, Capacitor_SMD:C_0603_1608Metric_Pad1.08x0.95mm_HandSolder, F.Cu at (224.2, 46.1)
- added C2: 100nF, Capacitor_SMD:C_0603_1608Metric_Pad1.08x0.95mm_HandSolder, F.Cu at (219.9, 43.6)
- added C20: 100uF, easyeda2kicad:CAP-SMD_BD10.0-L10.3-W10.3-FD, F.Cu at (246.7, 45.6)
- added C21: 10uF, Capacitor_SMD:C_1206_3216Metric_Pad1.33x1.80mm_HandSolder, F.Cu at (262.2, 64.7)
- added C22: 100uF, easyeda2kicad:CAP-SMD_BD10.0-L10.3-W10.3-FD, F.Cu at (246.7, 57.2)
- added C3: 1uF, Capacitor_SMD:C_0603_1608Metric_Pad1.08x0.95mm_HandSolder, F.Cu at (219.9, 46.1)
- added C30: 10uF, Capacitor_SMD:C_1206_3216Metric_Pad1.33x1.80mm_HandSolder, F.Cu at (262.2, 68.0)
- added C4: 470pF, Capacitor_SMD:C_0603_1608Metric_Pad1.08x0.95mm_HandSolder, F.Cu at (219.9, 48.6)
- added C5: 10nF, Capacitor_SMD:C_0603_1608Metric_Pad1.08x0.95mm_HandSolder, F.Cu at (219.9, 51.1)
- added C6: 10nF, Capacitor_SMD:C_0603_1608Metric_Pad1.08x0.95mm_HandSolder, F.Cu at (219.9, 53.6)
- added C7: 22nF, Capacitor_SMD:C_0603_1608Metric_Pad1.08x0.95mm_HandSolder, F.Cu at (219.9, 56.1)
- added C8: 100nF, Capacitor_SMD:C_0603_1608Metric_Pad1.08x0.95mm_HandSolder, F.Cu at (219.9, 58.6)
- added C9: 22nF, Capacitor_SMD:C_0603_1608Metric_Pad1.08x0.95mm_HandSolder, F.Cu at (219.9, 61.1)
- added D1: AB510S, easyeda2kicad:ABS-SMD_L5.0-W4.4-P4.00-LS7.0-BL, F.Cu at (221.4, 84.5)
- added D2: AB510S, easyeda2kicad:ABS-SMD_L5.0-W4.4-P4.00-LS7.0-BL, F.Cu at (228.3, 84.5)
- added D3: SMAJ58A, easyeda2kicad:SMA_L4.3-W2.6-LS5.2-RD, F.Cu at (255.0, 82.1)
- added FB1: 30R, Inductor_SMD:L_0603_1608Metric_Pad1.05x0.95mm_HandSolder, F.Cu at (224.2, 48.6)
- added FB2: 300R, Inductor_SMD:L_0603_1608Metric_Pad1.05x0.95mm_HandSolder, F.Cu at (224.2, 51.1)
- added FB3: 300R, Inductor_SMD:L_0603_1608Metric_Pad1.05x0.95mm_HandSolder, F.Cu at (224.2, 53.6)
- added L1: G2401CE, easyeda2kicad:SMD-24_L15.1-W7.1-P1.00-LS10.0-BL, F.Cu at (225.9, 73.7)
- added L2: FC-SLF1065-251, easyeda2kicad:FILTER-SMD_L10.0-W8.7-FC-SLF1065-471, F.Cu at (259.6, 56.2)
- added L3: 68uH, easyeda2kicad:IND-SMD_L11.0-W10.2_CXP1050, F.Cu at (260.7, 45.4)
- added LED1: Yellow, easyeda2kicad:LED0603-RD, F.Cu at (236.2, 68.7)
- added LED2: Yellow, easyeda2kicad:LED0603-RD, F.Cu at (236.2, 71.4)
- added LED3: Yellow, easyeda2kicad:LED0603-RD, F.Cu at (236.2, 74.0)
- added LED4: Yellow, easyeda2kicad:LED0603-RD, F.Cu at (236.2, 76.7)
- added R1: 10R, Resistor_SMD:R_0603_1608Metric_Pad0.98x0.95mm_HandSolder, F.Cu at (224.2, 56.1)
- added R10: 10R, Resistor_SMD:R_0603_1608Metric_Pad0.98x0.95mm_HandSolder, F.Cu at (228.6, 51.1)
- added R11: 49R, Resistor_SMD:R_0603_1608Metric_Pad0.98x0.95mm_HandSolder, F.Cu at (228.6, 53.6)
- added R12: 49R, Resistor_SMD:R_0603_1608Metric_Pad0.98x0.95mm_HandSolder, F.Cu at (228.6, 56.1)
- added R13: 49R, Resistor_SMD:R_0603_1608Metric_Pad0.98x0.95mm_HandSolder, F.Cu at (228.6, 58.6)
- added R14: 49R, Resistor_SMD:R_0603_1608Metric_Pad0.98x0.95mm_HandSolder, F.Cu at (228.6, 61.1)
- added R15: 0R, Resistor_SMD:R_0603_1608Metric_Pad0.98x0.95mm_HandSolder, F.Cu at (228.6, 63.6)
- added R16: 75R, Resistor_SMD:R_0603_1608Metric_Pad0.98x0.95mm_HandSolder, F.Cu at (228.6, 66.2)
- added R17: 75R, Resistor_SMD:R_0603_1608Metric_Pad0.98x0.95mm_HandSolder, F.Cu at (232.9, 41.1)
- added R18: 75R, Resistor_SMD:R_0603_1608Metric_Pad0.98x0.95mm_HandSolder, F.Cu at (232.9, 43.6)
- added R19: 75R, Resistor_SMD:R_0603_1608Metric_Pad0.98x0.95mm_HandSolder, F.Cu at (232.9, 46.1)
- added R2: 12.1k, Resistor_SMD:R_0603_1608Metric_Pad0.98x0.95mm_HandSolder, F.Cu at (224.2, 58.6)
- added R20: 75R, Resistor_SMD:R_0603_1608Metric_Pad0.98x0.95mm_HandSolder, F.Cu at (232.9, 48.6)
- added R21: 75R, Resistor_SMD:R_0603_1608Metric_Pad0.98x0.95mm_HandSolder, F.Cu at (232.9, 51.1)
- added R22: 75R, Resistor_SMD:R_0603_1608Metric_Pad0.98x0.95mm_HandSolder, F.Cu at (232.9, 53.6)
- added R23: 75R, Resistor_SMD:R_0603_1608Metric_Pad0.98x0.95mm_HandSolder, F.Cu at (232.9, 56.1)
- added R24: 1.5k, Resistor_SMD:R_0603_1608Metric_Pad0.98x0.95mm_HandSolder, F.Cu at (232.9, 58.6)
- added R25: 24.9k, Resistor_SMD:R_0603_1608Metric_Pad0.98x0.95mm_HandSolder, F.Cu at (232.9, 61.1)
- added R26: 63.4, Resistor_SMD:R_0603_1608Metric_Pad0.98x0.95mm_HandSolder, F.Cu at (232.9, 63.6)
- added R27: 249R, Resistor_SMD:R_0603_1608Metric_Pad0.98x0.95mm_HandSolder, F.Cu at (232.9, 66.2)
- added R28: 49.9k, Resistor_SMD:R_0603_1608Metric_Pad0.98x0.95mm_HandSolder, F.Cu at (237.3, 41.1)
- added R29: 49.9k, Resistor_SMD:R_0603_1608Metric_Pad0.98x0.95mm_HandSolder, F.Cu at (237.3, 43.6)
- added R3: 33R, Resistor_SMD:R_0603_1608Metric_Pad0.98x0.95mm_HandSolder, F.Cu at (224.2, 61.1)
- added R30: 21k, Resistor_SMD:R_0603_1608Metric_Pad0.98x0.95mm_HandSolder, F.Cu at (237.3, 46.1)
- added R31: 21k, Resistor_SMD:R_0603_1608Metric_Pad0.98x0.95mm_HandSolder, F.Cu at (237.3, 48.6)
- added R32: 21k, Resistor_SMD:R_0603_1608Metric_Pad0.98x0.95mm_HandSolder, F.Cu at (237.3, 51.1)
- added R33: 249k, Resistor_SMD:R_0603_1608Metric_Pad0.98x0.95mm_HandSolder, F.Cu at (237.3, 53.6)
- added R34: 36.5k, Resistor_SMD:R_0603_1608Metric_Pad0.98x0.95mm_HandSolder, F.Cu at (237.3, 56.1)
- added R35: 348k, Resistor_SMD:R_0603_1608Metric_Pad0.98x0.95mm_HandSolder, F.Cu at (237.3, 58.6)
- added R36: 12k, Resistor_SMD:R_0603_1608Metric_Pad0.98x0.95mm_HandSolder, F.Cu at (237.3, 61.1)
- added R37: 1.5k, Resistor_SMD:R_0603_1608Metric_Pad0.98x0.95mm_HandSolder, F.Cu at (237.3, 63.6)
- added R38: 1k, Resistor_SMD:R_0603_1608Metric_Pad0.98x0.95mm_HandSolder, F.Cu at (237.3, 66.2)
- added R4: 10k, Resistor_SMD:R_0603_1608Metric_Pad0.98x0.95mm_HandSolder, F.Cu at (224.2, 63.6)
- added R5: 1.5k, Resistor_SMD:R_0603_1608Metric_Pad0.98x0.95mm_HandSolder, F.Cu at (224.2, 66.2)
- added R6: 1.5k, Resistor_SMD:R_0603_1608Metric_Pad0.98x0.95mm_HandSolder, F.Cu at (228.6, 41.1)
- added R7: 1.5k, Resistor_SMD:R_0603_1608Metric_Pad0.98x0.95mm_HandSolder, F.Cu at (228.6, 43.6)
- added R8: 1.5k, Resistor_SMD:R_0603_1608Metric_Pad0.98x0.95mm_HandSolder, F.Cu at (228.6, 46.1)
- added R9: 10R, Resistor_SMD:R_0603_1608Metric_Pad0.98x0.95mm_HandSolder, F.Cu at (228.6, 48.6)
- added RJ1: R-RJ45R08P-C000, easyeda2kicad:RJ45-TH_R-RJ45R08P-C000, F.Cu at (249.3, 68.2)
- added TP3: GNDREF, TestPoint:TestPoint_Pad_D2.0mm, F.Cu at (241.5, 82.2)
- added TP4: VCOM, TestPoint:TestPoint_Pad_D2.0mm, F.Cu at (241.5, 86.2)
- added U1: LAN8720A, easyeda2kicad:QFN-24_L4.0-W4.0-P0.50-BL-EP2.6, F.Cu at (261.9, 72.5)
- added U2: TPS2372-4RGWR, easyeda2kicad:VQFN-20_L5.0-W5.0-P0.65-BL-EP2.2, F.Cu at (262.1, 83.6)
- added U3: TPS54560DDAR, easyeda2kicad:SOIC-8_L5.0-W4.0-P1.27-LS6.0-BL-EP2.0, F.Cu at (234.8, 84.3)
- added U4: SS510, easyeda2kicad:SMB_L4.3-W3.6-LS5.3-RD, F.Cu at (247.4, 82.6)
- added U6: TLV75533PDBVR, easyeda2kicad:SOT-23-5_L3.0-W1.7-P0.95-LS2.8-BR, F.Cu at (261.5, 77.7)
- TP1: value VDD -> 24V_OUT
- TP2: value GND -> GND_OUT
Connections:
- TP1 pad 1: VDD -> Net-(C21-Pad1)
- TP2 pad 1: GND -> IRSHDL_EN

Commit message: updates
Parts:
- added C17: 100nF, Capacitor_SMD:C_0603_1608Metric_Pad1.08x0.95mm_HandSolder, F.Cu at (153.8, 164.9)
- added C18: 1nF, Capacitor_SMD:C_0603_1608Metric_Pad1.08x0.95mm_HandSolder, F.Cu at (153.8, 148.1)
- added C19: 1nF, Capacitor_SMD:C_0603_1608Metric_Pad1.08x0.95mm_HandSolder, F.Cu at (153.9, 160.3)
- moved C20 150.8 mm to (164.0, 171.7), turned to -90 degrees
- moved L2 144.2 mm to (153.9, 154.1), turned to 90 degrees
- moved RJ1 143.8 mm to (115.8, 121.7), turned to -90 degrees
- moved U2 140.0 mm to (153.4, 171.9), turned to 180 degrees
- moved R17 132.4 mm to (145.2, 140.2), turned to 180 degrees
- moved D3 129.3 mm to (153.8, 162.7), turned to 180 degrees
- moved R18 128.1 mm to (145.2, 137.0), turned to 180 degrees
- moved TP3 126.0 mm to (164.0, 181.5)
- moved C12 122.2 mm to (148.6, 137.0)
- moved R19 121.4 mm to (145.4, 130.1), turned to 180 degrees
- moved R16 116.3 mm to (145.2, 147.2), turned to 180 degrees
- moved C13 114.9 mm to (148.7, 130.1)
- moved L1 110.0 mm to (136.4, 137.6), turned to 90 degrees
- moved C10 109.8 mm to (148.6, 147.2)
- moved TP4 109.0 mm to (164.0, 162.9)
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Connections:
- net IRSHDL_EN renamed GNDREF
- net MPS_DUTY renamed GND2
Routing:
- net 4 TC: track 0.00 -> 67.2 mm, vias 0 -> 2
- net Net-(L1-Pad2): track 0.00 -> 41.4 mm
- net Net-(L1-Pad3): track 0.00 -> 41.4 mm
- net Net-(L1-Pad5): track 0.00 -> 40.7 mm
- net Net-(L1-Pad6): track 0.00 -> 40.7 mm
- net Net-(L1-Pad9): track 0.00 -> 39.3 mm, vias 0 -> 1
- net Net-(L1-Pad8): track 0.00 -> 39.3 mm, vias 0 -> 1
- net Net-(L1-Pad12): track 0.00 -> 37.4 mm, vias 0 -> 1
- net Net-(L1-Pad11): track 0.00 -> 37.4 mm
- net 7 NC: track 0.00 -> 32.8 mm
- net 8 GND: track 0.00 -> 32.8 mm, vias 0 -> 2
- net 6 RD-: track 0.00 -> 32.2 mm
- net 3 RD+: track 0.00 -> 32.2 mm
- net 1 TD+: track 0.00 -> 31.6 mm
- net 2 TD-: track 0.00 -> 31.6 mm
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
Commit message: update stuff a little bit
Parts:
- moved C1 203.8 mm to (17.4, 17.4)
- moved C2 203.8 mm to (17.4, 19.9)
- moved C3 203.8 mm to (17.4, 22.4)
- moved C4 203.8 mm to (17.4, 24.9)
- moved C5 203.8 mm to (17.4, 27.4)
- moved C6 203.8 mm to (17.4, 29.9)
- moved C7 203.8 mm to (17.4, 32.5)
- moved C8 203.8 mm to (17.4, 35.0)
- moved C9 203.8 mm to (17.4, 37.5)
- moved FB1 203.8 mm to (21.8, 24.9)
- moved R1 203.8 mm to (21.8, 32.5)
- moved R10 203.8 mm to (26.1, 27.4)
- moved R2 203.8 mm to (21.8, 35.0)
- moved R3 203.8 mm to (21.8, 37.5)
- moved R4 203.8 mm to (21.8, 40.0)
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Routing:
- net GND: vias 289 -> 282

Commit message: update
Parts:
- added C23: 2.2uF, Capacitor_SMD:C_0805_2012Metric_Pad1.18x1.45mm_HandSolder, F.Cu at (239.2, 92.6)
- moved C1 190.7 mm to (130.5, 171.0)
- moved FB1 183.4 mm to (141.8, 163.6), turned to 90 degrees
- moved C2 183.2 mm to (129.5, 164.8), turned to 90 degrees
- moved R8 182.7 mm to (122.5, 177.7), turned to -90 degrees
- moved R9 182.5 mm to (126.0, 177.7), turned to 90 degrees
- moved C3 182.3 mm to (116.0, 175.7), turned to 180 degrees
- moved C4 178.7 mm to (116.0, 174.0), turned to 180 degrees
- moved C7 178.3 mm to (138.3, 163.6), turned to -90 degrees
- moved C8 177.7 mm to (140.0, 163.6), turned to -90 degrees
- moved R10 176.5 mm to (118.8, 177.7), turned to 90 degrees
- moved R1 175.6 mm to (120.5, 177.7), turned to 90 degrees
- moved C5 175.1 mm to (116.0, 172.2), turned to 180 degrees
- moved C6 169.4 mm to (116.0, 167.7), turned to 180 degrees
- moved R4 168.9 mm to (130.5, 169.2)
- moved C9 163.2 mm to (129.0, 156.5), turned to -90 degrees
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Routing:
- net 1 TD+: track 31.6 -> 17.1 mm
- net 2 TD-: track 31.6 -> 17.5 mm
- net 4 TC: track 67.2 -> 53.9 mm, vias 2 -> 0
- net 3 RD+: track 32.2 -> 20.1 mm
- net VDDCR: track 0.00 -> 11.1 mm
- net 6 RD-: track 32.2 -> 21.6 mm
- net +3V3_LAN: track 0.00 -> 10.1 mm, vias 0 -> 1
- net IO18 PHY_MDIO: track 0.00 -> 7.74 mm
- net Net-(U1-~{RST}): track 0.00 -> 6.89 mm
- net Net-(U1-RBIAS): track 0.00 -> 6.45 mm
- net 7 NC: track 32.8 -> 26.7 mm
- net Net-(U1-RXD1/MODE1): track 0.00 -> 5.99 mm
- net Net-(U1-RXD0/MODE0): track 0.00 -> 5.47 mm
- net Net-(U1-CRS_DV/MODE2): track 0.00 -> 5.19 mm
- net Net-(U1-RXER/PHYAD0): track 0.00 -> 5.05 mm
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
Commit message: more
Parts:
- removed TP3: GNDREF, TestPoint:TestPoint_Pad_D2.0mm
- removed TP4: VCOM, TestPoint:TestPoint_Pad_D2.0mm
- added C15: 1uF, Capacitor_SMD:C_0603_1608Metric_Pad1.08x0.95mm_HandSolder, B.Cu at (97.0, 147.1)
- added C16: 1uF, Capacitor_SMD:C_0603_1608Metric_Pad1.08x0.95mm_HandSolder, B.Cu at (93.9, 143.8)
- added C24: 2.2uF, Capacitor_SMD:C_0805_2012Metric_Pad1.18x1.45mm_HandSolder, F.Cu at (156.6, 121.7)
- added C25: 2.2uF, Capacitor_SMD:C_0805_2012Metric_Pad1.18x1.45mm_HandSolder, F.Cu at (158.7, 121.7)
- added C26: 3.3nF, Capacitor_SMD:C_0603_1608Metric_Pad1.08x0.95mm_HandSolder, F.Cu at (176.4, 123.9)
- added C27: 3.3nF, Capacitor_SMD:C_0603_1608Metric_Pad1.08x0.95mm_HandSolder, F.Cu at (174.6, 123.9)
- added C28: 100nF, Capacitor_SMD:C_0603_1608Metric_Pad1.08x0.95mm_HandSolder, F.Cu at (163.6, 120.5)
- C1, C14, C2, C3, C4, C5, C6, C7, C8, C9, FB1, LED4, R1, R10, R11, R12, R13, R14, R15, R2, R24, R3, R37, R38, R4, R5, R6, R7, R8, R9, U1, U6: moved to B.Cu
- moved U6 178.1 mm to (96.5, 144.8), turned to 180 degrees
- moved C14 164.1 mm to (92.4, 143.8), turned to -90 degrees
- moved R37 164.0 mm to (97.0, 148.6), turned to 180 degrees
- moved LED4 157.3 mm to (97.0, 150.1), turned to 180 degrees
- moved R20 133.2 mm to (107.6, 93.8)
- moved U3 132.8 mm to (168.6, 123.7), turned to -90 degrees
- moved R21 131.4 mm to (107.6, 90.8)
- moved R22 129.9 mm to (107.6, 87.8)
- moved R23 128.5 mm to (107.6, 84.7)
- moved L3 112.9 mm to (171.3, 114.4), turned to 90 degrees
- moved R32 112.2 mm to (146.0, 116.4), turned to 180 degrees
- moved R31 112.1 mm to (146.0, 113.8), turned to 180 degrees
- moved R30 112.0 mm to (146.0, 111.1), turned to 180 degrees
- moved FB2 110.9 mm to (127.2, 104.9), turned to -90 degrees
- moved R29 110.8 mm to (163.6, 126.4), turned to 90 degrees
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Routing:
- net 2 TD-: track 17.5 -> 35.7 mm, vias 0 -> 1
- net 1 TD+: track 17.1 -> 34.8 mm, vias 0 -> 1
- net Net-(C21-Pad1): track 0.00 -> 16.2 mm
- net 3 RD+: track 20.1 -> 34.3 mm, vias 0 -> 1
- net 6 RD-: track 21.6 -> 34.9 mm, vias 0 -> 1
- net Net-(U3-FB): track 0.00 -> 11.3 mm
- net Net-(U3-COMP): track 0.00 -> 5.31 mm
- net GND: track 3.04 -> 0.00 mm, vias 229 -> 225
- net Net-(U3-EN): track 0.00 -> 2.65 mm
- net Net-(L1-Pad21): track 2.31 -> 0.00 mm
- net Net-(L1-Pad18): track 2.30 -> 0.01 mm
- net Net-(L1-Pad24): track 2.31 -> 0.05 mm
- net Net-(L1-Pad15): track 2.32 -> 0.10 mm
- net Net-(C26-Pad1): track 0.00 -> 1.84 mm
- net Net-(U3-RT/CLK): track 0.00 -> 1.70 mm
- removed copper zone on B.Cu, net GND
- removed copper zone on F.Cu, net GND
- removed copper zone on In1.Cu, net GND
- removed copper zone on In2.Cu, net GND
Other:
- board size 34.2 x 70.7 mm -> 120 x 72 mm
- board text removed: "Janek"
- board text removed: "github.com/janekc"
