File: QuinledPoEHat/QuinledPoEHat.kicad_sch (KiCad schematic)
At the start: 5 parts, among them U1 QuinLED-ESP32, U2 TPS2372-3RGWR

Commit message: update
Parts:
- removed RJ1: RJ-055-1, easyeda2kicad:RJ45-SMD_RJ-055-1, symbol easyeda2kicad:RJ-055-1
- removed U1: QuinLED-ESP32, quinled:QuinLED-ESP32, symbol quinled:QuinLED-ESP32
- added C1, C14, C2, C8: 100nF, Capacitor_SMD:C_0603_1608Metric_Pad1.08x0.95mm_HandSolder, symbol Device:C
- added C10, C11, C12, C13, C5, C6: 10nF, Capacitor_SMD:C_0603_1608Metric_Pad1.08x0.95mm_HandSolder, symbol Device:C
- added C15, C16: 1uF, symbol Device:C
- added C17: 100nF, symbol Device:C
- added C18, C19: 1nF, symbol Device:C
- added C3: ?1u1R, Capacitor_SMD:C_0603_1608Metric_Pad1.08x0.95mm_HandSolder, symbol Device:C
- added C4: 470pF, Capacitor_SMD:C_0603_1608Metric_Pad1.08x0.95mm_HandSolder, symbol Device:C
- added C7, C9: 22nF, Capacitor_SMD:C_0603_1608Metric_Pad1.08x0.95mm_HandSolder, symbol Device:C
- added D1, D2: AB510S, easyeda2kicad:ABS-SMD_L5.0-W4.4-P4.00-LS7.0-BL, symbol easyeda2kicad:AB510S
- added D3: SMAJ58A, easyeda2kicad:SMA_L4.3-W2.6-LS5.2-RD, symbol easyeda2kicad:SMAJ58A-C151246
- added FB1: 30R, Inductor_SMD:L_0603_1608Metric_Pad1.05x0.95mm_HandSolder, symbol Device:FerriteBead_Small
- added FB2, FB3: 300R, Inductor_SMD:L_0603_1608Metric_Pad1.05x0.95mm_HandSolder, symbol Device:FerriteBead_Small
- added L1: G2401CE, easyeda2kicad:SMD-24_L15.1-W7.1-P1.00-LS10.0-BL, symbol easyeda2kicad:G2401CE
- added L2: FC-SLF1065-251, easyeda2kicad:FILTER-SMD_L10.0-W8.7-FC-SLF1065-471, symbol easyeda2kicad:FC-SLF1065-251
- added R1, R10, R9: 10R, Resistor_SMD:R_0603_1608Metric_Pad0.98x0.95mm_HandSolder, symbol Device:R
- added R11, R12, R13, R14: 49R, Resistor_SMD:R_0603_1608Metric_Pad0.98x0.95mm_HandSolder, symbol Device:R
- added R15: 0R, Resistor_SMD:R_0603_1608Metric_Pad0.98x0.95mm_HandSolder, symbol Device:R
- added R16, R17, R18, R19, R20, R21, R22, R23: 75R, Resistor_SMD:R_0603_1608Metric_Pad0.98x0.95mm_HandSolder, symbol Device:R
- added R2: 12.1k, Resistor_SMD:R_0603_1608Metric_Pad0.98x0.95mm_HandSolder, symbol Device:R
- added R24, R5, R6, R7, R8: 1.5k, Resistor_SMD:R_0603_1608Metric_Pad0.98x0.95mm_HandSolder, symbol Device:R
- added R3: 33R, Resistor_SMD:R_0603_1608Metric_Pad0.98x0.95mm_HandSolder, symbol Device:R
- added R4: 10k, Resistor_SMD:R_0603_1608Metric_Pad0.98x0.95mm_HandSolder, symbol Device:R
- added RJ1: R-RJ45R08P-C000, easyeda2kicad:RJ45-TH_R-RJ45R08P-C000, symbol easyeda2kicad:R-RJ45R08P-C000
- added U1: LAN8720A, easyeda2kicad:QFN-24_L4.0-W4.0-P0.50-BL-EP2.6, symbol Interface_Ethernet:LAN8720A
- added U5: QuinLED-ESP32, symbol testown:QuinLED-ESP32-Ethernet-Hat
- added U6: TLV75533PDBVR, easyeda2kicad:SOT-23-5_L3.0-W1.7-P0.95-LS2.8-BR, symbol easyeda2kicad:TLV75533PDBVR
Connections:
- net GND: now also C1.2, C10.2, C11.2, C12.2, C13.2, C15.2, C16.2, C2.2, C3.2, C4.2, C5.2, C6.2, C7.2, C8.2, C9.2, R15.1, R2.2, R20.1, R21.1, R22.1, R23.1, U1.25 (VSS), U6.2 (GND)
- new net: C10.1, R16.1
- new net: L1.24, R20.2
- new net: C17.1, C19.1, D3.1 (C), FB3.1, L2.1
- new net: C17.2, C19.2, D3.2 (A), FB2.2, L2.4
- new net: L1.11, RJ1.7
- new net: L1.12, RJ1.8
- new net: L1.15, R23.2
- new net: L1.18, R22.2
- new net: L1.2, RJ1.1
- new net: L1.21, R21.2
- new net: L1.3, RJ1.2
- new net: L1.5, RJ1.3
- new net: L1.6, RJ1.6
- new net: L1.8, RJ1.4
- new net: L1.9, RJ1.5
- new net: C12.1, R18.1
- new net: R3.2, U1.5 (XTAL1/CLKIN)
- new net: C1.1, R4.2, U1.15 (~{RST})
- new net: C11.1, R17.1
- new net: C13.1, R19.1
- new net: R7.2, RJ1.11 (R+)
- new net: R9.2, U1.11 (CRS_DV/MODE2)
- new net: R2.1, U1.24 (RBIAS)
- new net: R8.1, U1.10 (RXER/PHYAD0)
- new net: R10.2, U1.7 (RXD1/MODE1)
- new net: R1.2, U1.8 (RXD0/MODE0)
- new net: R24.1, RJ1.10 (L-)
- new net +3.3VA: C6.1, C7.1, C8.1, C9.1, FB1.2, L1.16, L1.17, R11.2, R12.2, R13.2, R14.2, RJ1.9 (L+), U1.1 (VDD2A), U1.19 (VDD1A)
- new net +3V3_LAN: C15.1, C2.1, FB1.1, R4.1, R5.1, R6.1, R8.2, U1.9 (VDDIO), U6.5 (OUT)
- new net +48V: C18.1, D1.1 (+), D2.1 (+), FB3.2, L2.2
- new net +5V: C14.1, C16.1, U5.9 (5vF*), U6.1 (IN), U6.3 (EN)
- new net -48V: C18.2, D1.2 (-), D2.2 (-), FB2.1, L2.3
- new net 1 TD+: L1.23, R13.1, U1.21 (TXP)
- new net 2 TD-: L1.22, R12.1, U1.20 (TXN)
- new net 3 RD+: L1.20, R11.1, U1.23 (RXP)
- new net 6 RD-: L1.19, R14.1, U1.22 (RXN)
- new net 7 NC: L1.14
- new net ACTLED: R7.1, U1.3 (LED1/REGOFF)
- new net GND1: L1.13, R15.2, RJ1.12 (R-), RJ1.13 (S), RJ1.14 (S)
- new net IO17 CLK: R3.1, U5.23 (IO17)
- new net IO18 PHY_MDIO: R5.2, U1.12 (MDIO), U5.13 (IO18)
- new net IO19 TXD[0]: U1.17 (TXD0), U5.14 (IO19)
- new net IO21 TX_EN: U1.16 (TXEN), U5.22 (IO21)
- new net IO22 TXD[1]: U1.18 (TXD1), U5.21 (IO22)
- new net IO23 PHY_MDC: U1.13 (MDC), U5.15 (IO23)
- new net IO25 RXD[0]: R1.1, U5.30 (IO25)
- new net IO26 RXD[1]: R10.1, U5.12 (IO26)
- new net IO27 CRS_DV: R6.2, R9.1, U5.29 (IO27)
- new net IO5 EN: U5.16 (IO5)
- new net LINKLED: R24.2, U1.2 (LED2/~{INTSEL})
- new net PAIR12: D1.4, L1.1, R16.2
- new net PAIR36: D1.3, L1.4, R17.2
- new net PAIR45: D2.4, L1.7, R18.2
- new net PAIR78: D2.3, L1.10, R19.2
- new net VDDCR: C3.1, C4.1, C5.1, U1.6 (VDDCR)
- no-connect marks 10 -> 3
Other:
- note added: "LAN8720A Bootstrap pins: PHYAD0 = 1 MODE[2:0] = 111 (MCU needs to pull MODE[01] high) REGOFF = 0 = enable 1.2V internal regulator nINTSEL = 1 = external clock"
- moved on the sheet: TP1, TP2, U2

Commit message: update lcsc bestellt
Parts:
- removed U2: TPS2372-3RGWR, easyeda2kicad:VQFN-20_L5.0-W5.0-P0.65-BL-EP2.2, symbol easyeda2kicad:TPS2372-3RGWR
- added C20, C22: 100uF, easyeda2kicad:CAP-SMD_BD10.0-L10.3-W10.3-FD, symbol Device:C_Polarized_US
- added C21, C30: 10uF, Capacitor_SMD:C_1206_3216Metric_Pad1.33x1.80mm_HandSolder, symbol Device:C
- added C23, C24, C25: 2.2uF, symbol Device:C
- added C26, C27: 3.3nF, symbol Device:C
- added C28: 100nF, symbol Device:C
- added L3: 68uH, easyeda2kicad:IND-SMD_L11.0-W10.2_CXP1050, symbol easyeda2kicad:CXP1050-680M-AG(68UH)
- added LED1, LED2, LED3, LED4: Yellow, easyeda2kicad:LED0603-RD, symbol easyeda2kicad:LTST-C190GKT
- added R25: 24.9k, Resistor_SMD:R_0603_1608Metric_Pad0.98x0.95mm_HandSolder, symbol Device:R
- added R26: 63.4, Resistor_SMD:R_0603_1608Metric_Pad0.98x0.95mm_HandSolder, symbol Device:R
- added R27: 249R, Resistor_SMD:R_0603_1608Metric_Pad0.98x0.95mm_HandSolder, symbol Device:R
- added R28, R29: 49.9k, Resistor_SMD:R_0603_1608Metric_Pad0.98x0.95mm_HandSolder, symbol Device:R
- added R30, R31, R32: 21k, Resistor_SMD:R_0603_1608Metric_Pad0.98x0.95mm_HandSolder, symbol Device:R
- added R33: 249k, Resistor_SMD:R_0603_1608Metric_Pad0.98x0.95mm_HandSolder, symbol Device:R
- added R34: 36.5k, Resistor_SMD:R_0603_1608Metric_Pad0.98x0.95mm_HandSolder, symbol Device:R
- added R35: 348k, Resistor_SMD:R_0603_1608Metric_Pad0.98x0.95mm_HandSolder, symbol Device:R
- added R36: 12k, Resistor_SMD:R_0603_1608Metric_Pad0.98x0.95mm_HandSolder, symbol Device:R
- added R37: 1.5k, Resistor_SMD:R_0603_1608Metric_Pad0.98x0.95mm_HandSolder, symbol Device:R
- added R38: 1k, Resistor_SMD:R_0603_1608Metric_Pad0.98x0.95mm_HandSolder, symbol Device:R
- added TP3: GNDREF, TestPoint:TestPoint_Pad_D2.0mm, symbol Connector:TestPoint
- added TP4: VCOM, TestPoint:TestPoint_Pad_D2.0mm, symbol Connector:TestPoint
- added U2: TPS2372-4RGWR, easyeda2kicad:VQFN-20_L5.0-W5.0-P0.65-BL-EP2.2, symbol easyeda2kicad:TPS2372-4RGWR
- added U3: TPS54560DDAR, easyeda2kicad:SOIC-8_L5.0-W4.0-P1.27-LS6.0-BL-EP2.0, symbol easyeda2kicad:TPS54560DDAR
- added U4: SS510, easyeda2kicad:SMB_L4.3-W3.6-LS5.3-RD, symbol easyeda2kicad:SS510-SMB
- C3: value ?1u1R -> 1uF
- TP1: value VDD -> 24V_OUT
- TP2: value GND -> GND_OUT
Connections:
- net +3V3_LAN: now also R37.1
- net GND: now also C14.2, U5.1 (GND), U5.2 (GND*), U5.25 (GND), U5.28 (GND), LED4.1 (-), R38.1; no longer C10.2, C11.2, C12.2, C13.2, TP2.1
- net GND1: now also C10.2, C11.2, C12.2, C13.2
- net VDDCR: now also R38.2
- net VCOM: now reaches C17.1, C19.1, D3.1 (C), FB3.1, L2.1
- net VCOM: now also C20.1, C23.1, C24.1, C25.1, R25.1, R30.1, R31.1, R32.1, TP4.1, U2.1 (VDD), U3.2 (VIN)
- net MPS_DUTY: now reaches C17.2, C19.2, D3.2 (A), FB2.2, L2.4
- net MPS_DUTY: now also R26.1, R27.1, R28.2, U2.21 (EP), U2.4 (VSS), U2.5 (VSS), U2.8 (AMPS_CTL), U2.9 (MPS_DUTY)
- net VDD: no longer names the net of TP1.1
- net VDD: now also C21.1, C22.1, C30.1, L3.2, R35.2
- new net: LED1.2 (+), R30.2
- new net: LED2.2 (+), R31.2
- new net: R29.2, U3.3 (EN)
- new net: R27.2, U2.6 (CLSB)
- new net: R33.2, U3.4 (RT/CLK)
- new net: C26.1, R34.1
- new net: C27.1, R34.2, U3.6 (COMP)
- new net: R25.2, U2.2 (DEN)
- new net: LED3.2 (+), R32.2
- new net: R26.2, U2.3 (CLSA)
- new net: R28.1, U2.7 (REF)
- new net: C28.2, L3.1, U3.8 (SW), U4.1
- new net: C28.1, U3.1 (BOOT)
- new net: R35.1, R36.2, U3.5 (FB)
- new net: LED4.2 (+), R37.2
- new net BT: LED3.1 (-)
- new net GNDREF: C20.2, C21.2, C22.2, C23.2, C24.2, C25.2, C26.2, C27.2, C30.2, R33.1, R36.1, TP2.1, TP3.1, U2.11 (RTN), U2.12 (RTN), U2.16 (IRSHDL_EN), U3.7 (GND), U3.9 (EP), U4.2
- new net PG: R29.1, U2.13 (PG)
- new net TPH: LED1.1 (-), U2.18 (TPH)
- new net TPL: LED2.1 (-), U2.17 (TPL)
- new net ~{BT}: U2.19 (~{BT})
- no-connect marks 3 -> 7
Other:
- note added: "Output to LedBrain 24V 3A"
- note added: "Pins used in the original ethernet extension board"
- note removed: "Output"
- note removed: "Pins used for the ethernet extension board (Do not use those)"
- moved on the sheet: C1, C10, C11, C12, C13, C15, C16, C17, C18, C19, C2, C3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

Commit message: updates
Parts:
- C17, C18, C19: footprint (none) -> Capacitor_SMD:C_0603_1608Metric_Pad1.08x0.95mm_HandSolder
- C23: footprint (none) -> Capacitor_SMD:C_0805_2012Metric_Pad1.18x1.45mm_HandSolder
Connections:
- net MPS_DUTY renamed GND2

Commit message: more
Parts:
- removed TP3: GNDREF, TestPoint:TestPoint_Pad_D2.0mm, symbol Connector:TestPoint
- removed TP4: VCOM, TestPoint:TestPoint_Pad_D2.0mm, symbol Connector:TestPoint
- C15, C16, C26, C27, C28: footprint (none) -> Capacitor_SMD:C_0603_1608Metric_Pad1.08x0.95mm_HandSolder
- C24, C25: footprint (none) -> Capacitor_SMD:C_0805_2012Metric_Pad1.18x1.45mm_HandSolder
- U5: footprint (none) -> quinled:QuinLED-ESP32-Ethernet-Hat
Changed lines of the file:
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@@
 	)
 	(symbol
-		(lib_id "Connector:TestPoint")
-		(at 185.42 220.98 180)
-		(unit 1)
-		(body_style 1)
-		(exclude_from_sim no)
-		(in_bom yes)
-		(on_board yes)
-		(in_pos_files yes)
-		(dnp no)
-		(fields_autoplaced yes)
-		(property "Reference" "TP4"
-			(at 187.96 223.0119 0)
-			(show_name no)
-			(do_not_autoplace no)
-			(effects
-				(font
-					(size 1.27 1.27)
-				)
-				(justify right)
-			)
-		)
-		(property "Value" "VCOM"
-			(at 187.96 225.5519 0)
-			(show_name no)
-			(do_not_autoplace no)
-			(effects
-				(font
-					(size 1.27 1.27)
-				)
-				(justify right)
-			)
-		)
-		(property "Footprint" "TestPoint:TestPoint_Pad_D2.0mm"
-			(at 180.34 220.98 0)
-			(hide yes)
-			(show_name no)
-			(do_not_autoplace no)
-			(effects
-				(font
-					(size 1.27 1.27)
-				)
-			)
-		)
-		(property "Datasheet" ""
-			(at 180.34 220.98 0)
-			(hide yes)
-			(show_name no)
-			(do_not_autoplace no)
-			(effects
-				(font
-					(size 1.27 1.27)
-				)
-			)
-		)
-		(property "Description" "test point"
-			(at 185.42 220.98 0)
-			(hide yes)
-			(show_name no)
-			(do_not_autoplace no)
-			(effects
-				(font
-					(size 1.27 1.27)
-				)
-			)
-		)
-		(pin "1"
-		)
-		(instances
-			(project "QuinledPoEHat"
-				(path "/bc40478d-6be8-4bd8-9e2c-1b79fb7d568e"
-					(reference "TP4")
-					(unit 1)
-				)
-			)
-		)
-	)
-	(symbol
 		(lib_id "Device:R")
 		(at 111.76 240.03 90)
@@
 	)
 	(symbol
-		(lib_id "Connector:TestPoint")
-		(at 185.42 247.65 0)
-		(unit 1)
-		(body_style 1)
-		(exclude_from_sim no)
-		(in_bom yes)
-		(on_board yes)
-		(in_pos_files yes)
-		(dnp no)
-		(fields_autoplaced yes)
-		(property "Reference" "TP3"
-			(at 187.96 243.0779 0)
-			(show_name no)
-			(do_not_autoplace no)
-			(effects
-				(font
-					(size 1.27 1.27)
-				)
-				(justify left)
-			)
-		)
-		(property "Value" "GNDREF"
-			(at 187.96 245.6179 0)
-			(show_name no)
-			(do_not_autoplace no)
-			(effects
-				(font
-					(size 1.27 1.27)
-				)
-				(justify left)
-			)
-		)
-		(property "Footprint" "TestPoint:TestPoint_Pad_D2.0mm"
-			(at 190.5 247.65 0)
-			(hide yes)
-			(show_name no)
-			(do_not_autoplace no)
-			(effects
-				(font
-					(size 1.27 1.27)
-				)
-			)
-		)
-		(property "Datasheet" ""
-			(at 190.5 247.65 0)
-			(hide yes)
-			(show_name no)
-			(do_not_autoplace no)
-			(effects
-				(font
-					(size 1.27 1.27)
-				)
-			)
-		)
-		(property "Description" "test point"
-			(at 185.42 247.65 0)
-			(hide yes)
-			(show_name no)
-			(do_not_autoplace no)
-			(effects
-				(font
-					(size 1.27 1.27)
-				)
-			)
-		)
-		(pin "1"
-		)
-		(instances
-			(project "QuinledPoEHat"
-				(path "/bc40478d-6be8-4bd8-9e2c-1b79fb7d568e"
-					(reference "TP3")
-					(unit 1)
-				)
-			)
-		)
-	)
-	(symbol
 		(lib_id "Device:C")
 		(at 246.38 238.76 0)
@@
 			)
 		)
-		(property "Footprint" ""
+		(property "Footprint" "Capacitor_SMD:C_0603_1608Metric_Pad1.08x0.95mm_HandSolder"
 			(at 247.3452 242.57 0)
 			(hide yes)
@@
 			)
 		)
-		(property "Footprint" ""
+		(property "Footprint" "Capacitor_SMD:C_0805_2012Metric_Pad1.18x1.45mm_HandSolder"
 			(at 209.2452 237.49 0)
 			(hide yes)
@@
 			)
 		)
-		(property "Footprint" ""
+		(property "Footprint" "Capacitor_SMD:C_0603_1608Metric_Pad1.08x0.95mm_HandSolder"
 			(at 238.4552 246.38 0)
 			(hide yes)
@@
 			)
 		)
-		(property "Footprint" ""
+		(property "Footprint" "quinled:QuinLED-ESP32-Ethernet-Hat"
 			(at 12.7 17.78 0)
 			(hide yes)
@@
 			)
 		)
-		(property "Footprint" ""
+		(property "Footprint" "Capacitor_SMD:C_0603_1608Metric_Pad1.08x0.95mm_HandSolder"
 			(at 287.02 213.6648 0)
 			(hide yes)
@@
 			)
 		)
-		(property "Footprint" ""
+		(property "Footprint" "Capacitor_SMD:C_0603_1608Metric_Pad1.08x0.95mm_HandSolder"
 			(at 219.4052 121.92 0)
 			(hide yes)
@@
 			)
 		)
-		(property "Footprint" ""
+		(property "Footprint" "Capacitor_SMD:C_0805_2012Metric_Pad1.18x1.45mm_HandSolder"
 			(at 220.6752 237.49 0)
 			(hide yes)
@@
 			)
 		)
-		(property "Footprint" ""
+		(property "Footprint" "Capacitor_SMD:C_0603_1608Metric_Pad1.08x0.95mm_HandSolder"
 			(at 180.0352 121.92 0)
 			(hide yes)
